File: PCB/arcade/arcade.kicad_pcb (KiCad board)
At the start: 2 copper layers, 254.8 x 58.3 mm, 17 parts, among them J1 USB_C_Receptacle_USB2.0_16P, J2 Conn_01x32_Pin, J3 Conn_01x32_Pin, J4 Conn_01x32_Pin, J5 Screw_Terminal_01x12, J6 Screw_Terminal_01x12, J7 Screw_Terminal_01x04, U1 ESP32-S3-WROOM-1, U2 TLC5947RHB, U3 TLC5947RHB, U4 TLC5947RHB, U5 ME6211C33M5

Commit message: pcb
Parts:
- moved J3 5.22 mm to (109.9, 73.3)
- moved J2 5.22 mm to (25.5, 73.3)
- moved J4 5.22 mm to (194.2, 73.3)
- moved U2 3.04 mm to (64.2, 84.1)
- moved U3 3.04 mm to (149.0, 84.1)
- moved U4 3.04 mm to (233.7, 84.1)
Routing:
- net Net-(J2-Pin_32): track 43.5 -> 0.00 mm
- net Net-(J3-Pin_32): track 43.1 -> 0.00 mm
- net Net-(J4-Pin_32): track 42.7 -> 0.00 mm
- net Net-(J4-Pin_2): track 40.8 -> 0.00 mm
- net Net-(J2-Pin_31): track 40.8 -> 0.00 mm
- net Net-(J3-Pin_2): track 40.4 -> 0.00 mm
- net Net-(J3-Pin_31): track 40.4 -> 0.00 mm
- net Net-(J4-Pin_31): track 40.0 -> 0.00 mm
- net Net-(J4-Pin_3): track 38.1 -> 0.00 mm
- net Net-(J2-Pin_30): track 38.0 -> 0.00 mm
- net Net-(J3-Pin_3): track 37.7 -> 0.00 mm
- net Net-(J3-Pin_30): track 37.6 -> 0.00 mm
- net Net-(J4-Pin_30): track 37.2 -> 0.00 mm
- net Net-(J4-Pin_4): track 35.3 -> 0.00 mm
- net Net-(J3-Pin_4): track 34.9 -> 0.00 mm
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Other:
- board size 254.8 x 58.3 mm -> 252.2 x 42.5 mm

Commit message: pcb
Parts:
- added C3: 22pf, Capacitor_SMD:C_0603_1608Metric_Pad1.08x0.95mm_HandSolder, F.Cu at (242.0, 134.7)
- added C4: 22pf, Capacitor_SMD:C_0603_1608Metric_Pad1.08x0.95mm_HandSolder, F.Cu at (242.0, 137.3)
- added C5: .01uf, Capacitor_SMD:C_0603_1608Metric_Pad1.08x0.95mm_HandSolder, F.Cu at (242.0, 139.8)
- added C7: .01uf, Capacitor_SMD:C_0603_1608Metric_Pad1.08x0.95mm_HandSolder, F.Cu at (242.0, 142.3)
- added FB2: FerriteBead, Inductor_SMD:L_0603_1608Metric, F.Cu at (250.7, 144.7)
- added R1: 22, Resistor_SMD:R_0603_1608Metric_Pad0.98x0.95mm_HandSolder, F.Cu at (242.0, 144.8)
- added R2: 22, Resistor_SMD:R_0603_1608Metric_Pad0.98x0.95mm_HandSolder, F.Cu at (242.0, 147.3)
- added R3: 10k, Resistor_SMD:R_0603_1608Metric_Pad0.98x0.95mm_HandSolder, F.Cu at (242.0, 149.8)
- added R6: 10k, Resistor_SMD:R_0603_1608Metric_Pad0.98x0.95mm_HandSolder, F.Cu at (242.0, 152.3)
- added U6: CD74HC4067M, Package_SO:SSOP-24_5.3x8.2mm_P0.65mm, F.Cu at (78.2, 97.3)
- added U7: CD74HC4067M, Package_SO:SSOP-24_5.3x8.2mm_P0.65mm, F.Cu at (132.3, 97.3)
- added U8: MAX3421EEHJ+T, max3421:21-0110-C_90-0149-32L_MXM, F.Cu at (248.9, 138.5)
- added Y1: Crystal_GND24, Crystal:Crystal_SMD_2520-4Pin_2.5x2.0mm, F.Cu at (246.4, 145.4)
- J6: value Screw_Terminal_01x12 -> Screw_Terminal_01x08; footprint TerminalBlock_Phoenix:TerminalBlock_Phoenix_MPT-0,5-12-2.54_1x12_P2.54mm_Horizontal -> TerminalBlock_Phoenix:TerminalBlock_Phoenix_MPT-0,5-8-2.54_1x08_P2.54mm_Horizontal
- J7: value Screw_Terminal_01x04 -> Screw_Terminal_01x12; footprint TerminalBlock_Phoenix:TerminalBlock_Phoenix_MPT-0,5-4-2.54_1x04_P2.54mm_Horizontal -> TerminalBlock_Phoenix:TerminalBlock_Phoenix_MPT-0,5-12-2.54_1x12_P2.54mm_Horizontal
- moved R4 18.1 mm to (38.9, 104.8), turned to -90 degrees
- moved J7 11.4 mm to (119.0, 107.7)
- moved R5 7.89 mm to (49.7, 102.4)
- moved J6 0.61 mm to (96.5, 107.7)
- moved J5 0.07 mm to (63.8, 107.7)
Connections:
- net Net-(J2-Pin_1) renamed /VBUS
- R4 pad 2: Net-(R4-Pad2) -> Net-(J1-SHIELD)
- R5 pad 2: Net-(R4-Pad2) -> Net-(J1-SHIELD)
- U1 pad 10: Net-(J5-Pin_7) -> unconnected-(U1-IO17-Pad10)
- U1 pad 11: Net-(J5-Pin_8) -> unconnected-(U1-IO18-Pad11)
- U1 pad 12: Net-(J5-Pin_9) -> unconnected-(U1-IO8-Pad12)
- U1 pad 15: Net-(J5-Pin_10) -> /IO3
- U1 pad 16: Net-(J5-Pin_11) -> /IO46
- U1 pad 17: Net-(J5-Pin_12) -> /IO9
- U1 pad 18: Net-(J6-Pin_1) -> /IO10
- U1 pad 19: Net-(J6-Pin_2) -> /IO11
- U1 pad 20: Net-(J6-Pin_3) -> /IO12
- U1 pad 21: Net-(J6-Pin_4) -> /IO13
- U1 pad 22: Net-(J6-Pin_5) -> /IO14
- U1 pad 23: Net-(J6-Pin_6) -> unconnected-(U1-IO21-Pad23)
- U1 pad 24: Net-(J7-Pin_1) -> unconnected-(U1-IO47-Pad24)
- U1 pad 26: Net-(J6-Pin_7) -> unconnected-(U1-IO45-Pad26)
- U1 pad 27: Net-(J7-Pin_2) -> unconnected-(U1-IO0-Pad27)
- U1 pad 29: Net-(J7-Pin_3) -> unconnected-(U1-IO36-Pad29)
- U1 pad 30: Net-(J7-Pin_4) -> unconnected-(U1-IO37-Pad30)
- U1 pad 31: Net-(J6-Pin_8) -> unconnected-(U1-IO38-Pad31)
- U1 pad 32: Net-(J6-Pin_9) -> unconnected-(U1-IO39-Pad32)
- U1 pad 33: Net-(J6-Pin_10) -> unconnected-(U1-IO40-Pad33)
- U1 pad 34: Net-(J6-Pin_11) -> unconnected-(U1-IO41-Pad34)
- U1 pad 35: Net-(J6-Pin_12) -> unconnected-(U1-IO42-Pad35)
- U1 pad 4: Net-(J5-Pin_1) -> unconnected-(U1-IO4-Pad4)
- U1 pad 5: Net-(J5-Pin_2) -> unconnected-(U1-IO5-Pad5)
- U1 pad 6: Net-(J5-Pin_3) -> unconnected-(U1-IO6-Pad6)
- U1 pad 7: Net-(J5-Pin_4) -> unconnected-(U1-IO7-Pad7)
- U1 pad 8: Net-(J5-Pin_5) -> /IO15
- U1 pad 9: Net-(J5-Pin_6) -> /IO16
Routing:
- net Net-(J7-Pin_4): track 111.8 -> 8.07 mm, vias 1 -> 0
- net Net-(J6-Pin_12): track 101.7 -> 0.00 mm
- net /IO46: track 0.00 -> 98.9 mm, vias 0 -> 4
- net /IO3: track 0.00 -> 98.3 mm, vias 0 -> 4
- net Net-(J6-Pin_11): track 97.8 -> 0.00 mm
- net Net-(J7-Pin_3): track 109.0 -> 12.8 mm, vias 1 -> 0
- net /IO11: track 0.00 -> 96.2 mm, vias 0 -> 2
- net /IO10: track 0.00 -> 95.5 mm, vias 0 -> 2
- net Net-(J6-Pin_10): track 93.6 -> 0.00 mm
- net /IO12: track 0.00 -> 91.4 mm
- net Net-(J7-Pin_2): track 105.7 -> 15.1 mm, vias 1 -> 0
- net Net-(J6-Pin_9): track 89.9 -> 0.00 mm
- net Net-(J7-Pin_1): track 98.1 -> 17.5 mm, vias 1 -> 0
- net Net-(J6-Pin_8): track 85.7 -> 23.2 mm
- net Net-(J6-Pin_7): track 74.5 -> 26.7 mm
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Other:
- board text added: "U6"

Commit message: stopping point on PCB
Parts:
- removed C3, C4: 22pf, Capacitor_SMD:C_0603_1608Metric_Pad1.08x0.95mm_HandSolder
- removed C5, C7: .01uf, Capacitor_SMD:C_0603_1608Metric_Pad1.08x0.95mm_HandSolder
- removed FB2: FerriteBead, Inductor_SMD:L_0603_1608Metric
- removed R1, R2: 22, Resistor_SMD:R_0603_1608Metric_Pad0.98x0.95mm_HandSolder
- removed R3, R6: 10k, Resistor_SMD:R_0603_1608Metric_Pad0.98x0.95mm_HandSolder
- removed Y1: Crystal_GND24, Crystal:Crystal_SMD_2520-4Pin_2.5x2.0mm
- added J10: USB_A, Connector_USB:USB_A_Molex_67643_Horizontal, F.Cu at (71.6, 99.3)
- added J11: USB_A, Connector_USB:USB_A_Molex_67643_Horizontal, F.Cu at (89.3, 99.3)
- added J12: Conn_01x06_Pin, Connector_PinHeader_2.54mm:PinHeader_1x06_P2.54mm_Horizontal, F.Cu at (138.0, 107.4)
- added J13: Conn_01x06_Pin, Connector_PinHeader_2.54mm:PinHeader_1x06_P2.54mm_Horizontal, F.Cu at (246.9, 107.4)
- added J14: Conn_01x04_Pin, Connector_PinHeader_2.54mm:PinHeader_1x04_P2.54mm_Vertical, F.Cu at (28.3, 80.1)
- added J8: Conn_01x03_Pin, Connector_PinHeader_2.54mm:PinHeader_1x03_P2.54mm_Horizontal, F.Cu at (120.5, 107.4)
- added J9: Conn_01x03_Pin, Connector_PinHeader_2.54mm:PinHeader_1x03_P2.54mm_Horizontal, F.Cu at (256.5, 107.4)
- added U9: FE1.1s, Package_SO:SSOP-28_3.9x9.9mm_P0.635mm, F.Cu at (52.2, 106.4)
- U8: value MAX3421EEHJ+T -> ATmega32U4-M; footprint max3421:21-0110-C_90-0149-32L_MXM -> Package_DFN_QFN:QFN-44-1EP_7x7mm_P0.5mm_EP5.2x5.2mm
- moved U8 192.7 mm to (60.8, 96.5)
- moved J5 80.5 mm to (144.3, 108.8)
- moved J6 80.5 mm to (177.0, 108.8)
- moved J7 80.5 mm to (199.5, 108.8)
- moved U6 80.5 mm to (158.8, 98.4)
- moved U7 80.5 mm to (212.9, 98.4)
- moved J1 16.8 mm to (30.1, 108.3)
- moved R5 16.8 mm to (32.9, 102.7)
- moved R4 11.6 mm to (27.4, 102.7), turned to 180 degrees
- moved C2 8.59 mm to (42.1, 105.7), turned to -90 degrees
- moved C1 7.25 mm to (39.3, 110.2), turned to 0 degrees
- moved C6 7.05 mm to (43.9, 105.7), turned to -90 degrees
- moved U5 6.08 mm to (39.0, 105.7), turned to 180 degrees
Connections:
- C1 pad 2: Net-(J1-SHIELD) -> /GND
- C2 pad 2: Net-(J1-SHIELD) -> /GND
- C6 pad 2: Net-(J1-SHIELD) -> /GND
- J1 pad A1: Net-(J1-SHIELD) -> /GND
- J1 pad A12: Net-(J1-SHIELD) -> /GND
- J1 pad B1: Net-(J1-SHIELD) -> /GND
- J1 pad B12: Net-(J1-SHIELD) -> /GND
- J1 pad S1: Net-(J1-SHIELD) -> /GND
- R4 pad 2: Net-(J1-SHIELD) -> /GND
- R5 pad 2: Net-(J1-SHIELD) -> /GND
- U1 pad 1: Net-(J1-SHIELD) -> /GND
- U1 pad 40: Net-(J1-SHIELD) -> /GND
- U1 pad 41: Net-(J1-SHIELD) -> /GND
- U2 pad 29: Net-(U2-GND) -> /GND
- U3 pad 29: Net-(U2-GND) -> /GND
- U4 pad 29: Net-(U2-GND) -> /GND
- U5 pad 2: Net-(J1-SHIELD) -> /GND
- U6 pad 12: unconnected-(U6-GND-Pad12) -> /GND
- U6 pad 24: unconnected-(U6-VCC-Pad24) -> /3.3v
- U7 pad 12: unconnected-(U7-GND-Pad12) -> /GND
- U7 pad 24: unconnected-(U7-VCC-Pad24) -> /3.3v
- U8 pad 12: Net-(U8-*RES) -> unconnected-(U8-PB7-Pad12)
- U8 pad 13: /IO12 -> unconnected-(U8-~{RESET}-Pad13)
- U8 pad 14: /IO10 -> /VCC
- U8 pad 15: /IO13 -> /GND
- U8 pad 16: /IO11 -> unconnected-(U8-XTAL2-Pad16)
- U8 pad 18: Net-(U8-INT) -> unconnected-(U8-PD0-Pad18)
- U8 pad 19: Net-(C7-Pad2) -> unconnected-(U8-PD1-Pad19)
- U8 pad 2: /3.3v -> unconnected-(U8-UVCC-Pad2)
- U8 pad 20: Net-(U8-D-) -> unconnected-(U8-PD2-Pad20)
- U8 pad 21: Net-(U8-D+) -> unconnected-(U8-PD3-Pad21)
- U8 pad 22: Net-(U8-VBCOMP) -> unconnected-(U8-PD5-Pad22)
- U8 pad 23: /3.3v -> /GND
- U8 pad 24: Net-(U8-XI) -> Net-(U8-AVCC-Pad24)
- U8 pad 25: Net-(U8-XO) -> unconnected-(U8-PD4-Pad25)
- U8 pad 3: Net-(C7-Pad2) -> unconnected-(U8-D--Pad3)
Routing:
- net /3.3v: track 13.5 -> 111.9 mm, vias 0 -> 3
- net /VBUS: track 492.3 -> 545.8 mm, vias 2 -> 6
- net Net-(J2-Pin_32): track 0.00 -> 42.8 mm
- net Net-(J3-Pin_32): track 0.00 -> 42.4 mm
- net Net-(J4-Pin_32): track 0.00 -> 42.0 mm
- net Net-(J2-Pin_31): track 0.00 -> 40.0 mm
- net Net-(J4-Pin_2): track 0.00 -> 39.7 mm
- net Net-(J3-Pin_31): track 0.00 -> 39.6 mm
- net Net-(J3-Pin_2): track 0.00 -> 39.3 mm
- net Net-(J4-Pin_31): track 0.00 -> 39.2 mm
- net Net-(J2-Pin_30): track 0.00 -> 37.3 mm
- net Net-(J4-Pin_3): track 0.00 -> 37.0 mm
- net Net-(J3-Pin_30): track 0.00 -> 36.9 mm
- net Net-(J3-Pin_3): track 0.00 -> 36.6 mm
- net Net-(J4-Pin_30): track 0.00 -> 36.5 mm
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- added copper zone on B.Cu, net /GND
Other:
- board size 252.2 x 42.5 mm -> 252.2 x 44.8 mm

Commit message: board
Parts:
- removed J12, J13: Conn_01x06_Pin, Connector_PinHeader_2.54mm:PinHeader_1x06_P2.54mm_Horizontal
- removed J14: Conn_01x04_Pin, Connector_PinHeader_2.54mm:PinHeader_1x04_P2.54mm_Vertical
- added C10: 22pf, Capacitor_SMD:C_0603_1608Metric_Pad1.08x0.95mm_HandSolder, F.Cu at (63.7, 93.9)
- added C11: 22pf, Capacitor_SMD:C_0603_1608Metric_Pad1.08x0.95mm_HandSolder, F.Cu at (69.8, 98.3)
- added C12: 22pf, Capacitor_SMD:C_0603_1608Metric_Pad1.08x0.95mm_HandSolder, F.Cu at (86.2, 100.5)
- added C13: 22pf, Capacitor_SMD:C_0603_1608Metric_Pad1.08x0.95mm_HandSolder, F.Cu at (86.2, 102.0)
- added C14: 22pf, Capacitor_SMD:C_0603_1608Metric_Pad1.08x0.95mm_HandSolder, F.Cu at (63.6, 95.9)
- added C3: 22pf, Capacitor_SMD:C_0603_1608Metric_Pad1.08x0.95mm_HandSolder, F.Cu at (81.4, 95.9)
- added C4: 22pf, Capacitor_SMD:C_0603_1608Metric_Pad1.08x0.95mm_HandSolder, F.Cu at (78.9, 93.2)
- added C5: 22pf, Capacitor_SMD:C_0603_1608Metric_Pad1.08x0.95mm_HandSolder, F.Cu at (57.3, 105.5)
- added C7: 22pf, Capacitor_SMD:C_0603_1608Metric_Pad1.08x0.95mm_HandSolder, F.Cu at (50.2, 95.8)
- added C8: 22pf, Capacitor_SMD:C_0603_1608Metric_Pad1.08x0.95mm_HandSolder, F.Cu at (60.7, 102.2)
- added C9: 22pf, Capacitor_SMD:C_0603_1608Metric_Pad1.08x0.95mm_HandSolder, F.Cu at (60.7, 103.9)
- added D1: SK6812MINI-E, LED_SMD:LED_SK6812MINI_PLCC4_3.5x3.5mm_P1.75mm, F.Cu at (41.7, 92.3)
- added H1: MountingHole, MountingHole:MountingHole_2.5mm_Pad_TopBottom, F.Cu at (125.2, 105.3)
- added H2: MountingHole, MountingHole:MountingHole_2.5mm_Pad_TopBottom, F.Cu at (2.77, 2.77)
- added H2: MountingHole, MountingHole:MountingHole_3mm_Pad_TopBottom, F.Cu at (153.7, 79.9)
- added H3: MountingHole, MountingHole:MountingHole_3mm_Pad_TopBottom, F.Cu at (42.8, 82.7)
- added H3: MountingHole, MountingHole:MountingHole_2.5mm_Pad_TopBottom, F.Cu at (2.77, 9.32)
- added H4: MountingHole, MountingHole:MountingHole_3mm_Pad_TopBottom, F.Cu at (92.1, 79.9)
- added H4: MountingHole, MountingHole:MountingHole_2.5mm_Pad_TopBottom, F.Cu at (2.77, 15.9)
- added J15: Conn_02x24_Odd_Even, Connector_PinHeader_2.54mm:PinHeader_2x24_P2.54mm_Horizontal, F.Cu at (28.1, 73.4)
- added J16: Conn_02x24_Odd_Even, Connector_PinHeader_2.54mm:PinHeader_2x24_P2.54mm_Horizontal, F.Cu at (98.3, 73.3)
- added R6: 5.1k, Resistor_SMD:R_0603_1608Metric_Pad0.98x0.95mm_HandSolder, F.Cu at (51.1, 93.2)
- added R7: 5.1k, Resistor_SMD:R_0603_1608Metric_Pad0.98x0.95mm_HandSolder, F.Cu at (57.3, 102.5)
- added R8: 5.1k, Resistor_SMD:R_0603_1608Metric_Pad0.98x0.95mm_HandSolder, F.Cu at (57.3, 104.0)
- added R9: 5.1k, Resistor_SMD:R_0603_1608Metric_Pad0.98x0.95mm_HandSolder, F.Cu at (50.2, 100.8)
- added Y1: Crystal_GND24, Crystal:Crystal_SMD_2520-4Pin_2.5x2.0mm, F.Cu at (78.9, 95.9)
- added Y2: Crystal_GND24, Crystal:Crystal_SMD_2520-4Pin_2.5x2.0mm, F.Cu at (59.8, 92.6)
- J2: value Conn_01x32_Pin -> Conn_02x03_Odd_Even; footprint Connector_PinHeader_2.54mm:PinHeader_1x32_P2.54mm_Horizontal -> Connector_PinHeader_2.54mm:PinHeader_2x03_P2.54mm_Horizontal
- J3: value Conn_01x32_Pin -> Conn_02x06_Odd_Even; footprint Connector_PinHeader_2.54mm:PinHeader_1x32_P2.54mm_Horizontal -> Connector_PinHeader_2.54mm:PinHeader_2x06_P2.54mm_Horizontal
- J4: value Conn_01x32_Pin -> Screw_Terminal_01x02; footprint Connector_PinHeader_2.54mm:PinHeader_1x32_P2.54mm_Horizontal -> TerminalBlock_Phoenix:TerminalBlock_Phoenix_MKDS-3-2-5.08_1x02_P5.08mm_Horizontal
- J8: value Conn_01x03_Pin -> Conn_01x02_Pin; footprint Connector_PinHeader_2.54mm:PinHeader_1x03_P2.54mm_Horizontal -> Connector_PinHeader_2.54mm:PinHeader_1x02_P2.54mm_Vertical
- J9: value Conn_01x03_Pin -> Conn_01x06_Pin; footprint Connector_PinHeader_2.54mm:PinHeader_1x03_P2.54mm_Horizontal -> Connector_PinHeader_2.54mm:PinHeader_1x06_P2.54mm_Vertical
- moved J9 231.0 mm to (25.8, 96.4), turned to 0 degrees
- moved J2 135.6 mm to (161.2, 73.3)
- moved U4 106.8 mm to (127.0, 79.8)
- moved J8 96.6 mm to (28.7, 77.3)
- moved U7 68.9 mm to (144.0, 102.2)
- moved J5 61.7 mm to (82.7, 112.6)
- moved J6 61.7 mm to (115.4, 112.6)
- moved J7 61.7 mm to (138.0, 112.6)
- moved U6 61.7 mm to (97.2, 102.2)
- moved U3 59.5 mm to (92.5, 65.5)
- moved J11 56.2 mm to (35.5, 83.2), turned to -90 degrees
- moved J3 48.9 mm to (155.2, 91.6), turned to 0 degrees
- moved C1 44.2 mm to (82.4, 100.5)
- moved U5 43.4 mm to (82.3, 103.0), turned to 0 degrees
- moved C2 40.2 mm to (82.3, 105.5), turned to 180 degrees
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Connections:
- J1 pad A6: Net-(U1-USB_D+) -> /DU+
- J1 pad A7: Net-(U1-USB_D-) -> /DU-
- J1 pad B6: Net-(U1-USB_D+) -> /DU+
- J1 pad B7: Net-(U1-USB_D-) -> /DU-
- J10 pad 1: unconnected-(J10-VBUS-Pad1) -> /VBUS
- J10 pad 2: unconnected-(J10-D--Pad2) -> /D2-
- J10 pad 3: unconnected-(J10-D+-Pad3) -> /D2+
- J10 pad 4: unconnected-(J10-GND-Pad4) -> /GND
- J10 pad SH: unconnected-(J10-Shield-PadSH) -> /GND
- J11 pad 1: unconnected-(J11-VBUS-Pad1) -> /VBUS
- J11 pad 2: unconnected-(J11-D--Pad2) -> /D3-
- J11 pad 3: unconnected-(J11-D+-Pad3) -> /D3+
- J11 pad 4: unconnected-(J11-GND-Pad4) -> /GND
- J11 pad SH: unconnected-(J11-Shield-PadSH) -> /GND
- J2 pad 1: /VBUS -> /GND
- J2 pad 2: Net-(J2-Pin_2) -> /GND
- J2 pad 3: Net-(J2-Pin_3) -> /IO39
- J2 pad 4: Net-(J2-Pin_4) -> /IO38
- J2 pad 5: /VBUS -> /EXT_5V
- J2 pad 6: Net-(J2-Pin_6) -> /EXT_5V
- J3 pad 1: /VBUS -> /CS1
- J3 pad 10: Net-(J3-Pin_10) -> /3.3v
- J3 pad 11: Net-(J3-Pin_11) -> /GND
- J3 pad 12: Net-(J3-Pin_12) -> /GND
- J3 pad 2: Net-(J3-Pin_2) -> /CS2
- J3 pad 3: Net-(J3-Pin_3) -> /MISO
- J3 pad 4: Net-(J3-Pin_4) -> /MISO
- J3 pad 5: /VBUS -> /MOSI
- J3 pad 6: Net-(J3-Pin_6) -> /MOSI
- J3 pad 7: Net-(J3-Pin_7) -> /SCK
- J3 pad 8: Net-(J3-Pin_8) -> /SCK
- J3 pad 9: /VBUS -> /3.3v
- J4 pad 1: /VBUS -> /GND
- J4 pad 2: Net-(J4-Pin_2) -> /EXT_5V
- J8 pad 1: unconnected-(J8-Pin_1-Pad1) -> /EXT_5V
- J8 pad 2: unconnected-(J8-Pin_2-Pad2) -> /VBUS
- J9 pad 2: unconnected-(J9-Pin_2-Pad2) -> /RXD0
- J9 pad 3: unconnected-(J9-Pin_3-Pad3) -> /TXD0
- U1 pad 12: unconnected-(U1-IO8-Pad12) -> /IO8
- U1 pad 13: Net-(U1-USB_D-) -> /D1-
- U1 pad 14: Net-(U1-USB_D+) -> /D1+
- U1 pad 25: Net-(U1-IO48) -> unconnected-(U1-IO48-Pad25)
- U1 pad 31: unconnected-(U1-IO38-Pad31) -> /IO38
- U1 pad 32: unconnected-(U1-IO39-Pad32) -> /IO39
- U1 pad 33: unconnected-(U1-IO40-Pad33) -> /IO40
- U1 pad 34: unconnected-(U1-IO41-Pad34) -> /IO41
- U1 pad 35: unconnected-(U1-IO42-Pad35) -> /IO42
- U1 pad 36: unconnected-(U1-RXD0-Pad36) -> /RXD0
- U1 pad 37: unconnected-(U1-TXD0-Pad37) -> /TXD0
- U1 pad 38: Net-(U1-IO2) -> unconnected-(U1-IO2-Pad38)
- U1 pad 39: Net-(U1-IO1) -> unconnected-(U1-IO1-Pad39)
- U1 pad 4: unconnected-(U1-IO4-Pad4) -> /IO4
- U1 pad 5: unconnected-(U1-IO5-Pad5) -> /IO5
- U1 pad 6: unconnected-(U1-IO6-Pad6) -> /IO6
- U1 pad 7: unconnected-(U1-IO7-Pad7) -> /IO7
- U2 pad 1: Net-(J2-Pin_32) -> Net-(J15-Pin_34)
- U2 pad 10: Net-(J2-Pin_20) -> Net-(J15-Pin_37)
- U2 pad 11: Net-(J2-Pin_19) -> Net-(J15-Pin_35)
- U2 pad 12: Net-(J2-Pin_18) -> Net-(J15-Pin_33)
- U2 pad 13: Net-(J2-Pin_16) -> Net-(J15-Pin_29)
- U2 pad 14: Net-(J2-Pin_15) -> Net-(J15-Pin_27)
- U2 pad 15: Net-(J2-Pin_14) -> Net-(J15-Pin_25)
- U2 pad 16: Net-(J2-Pin_12) -> Net-(J15-Pin_21)
- U2 pad 17: Net-(J2-Pin_11) -> Net-(J15-Pin_19)
- U2 pad 18: Net-(J2-Pin_10) -> Net-(J15-Pin_17)
- U2 pad 19: Net-(J2-Pin_8) -> Net-(J15-Pin_13)
- U2 pad 2: Net-(J2-Pin_31) -> Net-(J15-Pin_36)
- U2 pad 20: Net-(J2-Pin_7) -> Net-(J15-Pin_11)
- U2 pad 21: Net-(J2-Pin_6) -> Net-(J15-Pin_9)
- U2 pad 22: Net-(J2-Pin_4) -> Net-(J15-Pin_5)
- U2 pad 23: Net-(J2-Pin_3) -> Net-(J15-Pin_3)
- U2 pad 24: Net-(J2-Pin_2) -> Net-(J15-Pin_1)
- U2 pad 26: Net-(U1-IO48) -> /IO40
- U2 pad 28: /VBUS -> /EXT_5V
- U2 pad 3: Net-(J2-Pin_30) -> Net-(J15-Pin_38)
- U2 pad 31: Net-(U1-IO2) -> /IO41
- U2 pad 32: Net-(U1-IO1) -> /IO42
- U2 pad 33: unconnected-(U2-PowerPAD-Pad33) -> /GND
- U2 pad 4: Net-(J2-Pin_28) -> Net-(J15-Pin_42)
- U2 pad 5: Net-(J2-Pin_27) -> Net-(J15-Pin_44)
- U2 pad 6: Net-(J2-Pin_26) -> Net-(J15-Pin_46)
- U2 pad 7: Net-(J2-Pin_24) -> Net-(J15-Pin_45)
- U2 pad 8: Net-(J2-Pin_23) -> Net-(J15-Pin_43)
- U2 pad 9: Net-(J2-Pin_22) -> Net-(J15-Pin_41)
- U3 pad 1: Net-(J3-Pin_32) -> Net-(J16-Pin_17)
- U3 pad 10: Net-(J3-Pin_20) -> Net-(J16-Pin_41)
- U3 pad 11: Net-(J3-Pin_19) -> Net-(J16-Pin_43)
- U3 pad 12: Net-(J3-Pin_18) -> Net-(J16-Pin_45)
- U3 pad 13: Net-(J3-Pin_16) -> Net-(J15-Pin_2)
- U3 pad 14: Net-(J3-Pin_15) -> Net-(J15-Pin_4)
- U3 pad 15: Net-(J3-Pin_14) -> Net-(J15-Pin_6)
- U3 pad 16: Net-(J3-Pin_12) -> Net-(J15-Pin_10)
- U3 pad 17: Net-(J3-Pin_11) -> Net-(J15-Pin_12)
- U3 pad 18: Net-(J3-Pin_10) -> Net-(J15-Pin_14)
- U3 pad 19: Net-(J3-Pin_8) -> Net-(J15-Pin_18)
- U3 pad 2: Net-(J3-Pin_31) -> Net-(J16-Pin_19)
- U3 pad 20: Net-(J3-Pin_7) -> Net-(J15-Pin_20)
- U3 pad 21: Net-(J3-Pin_6) -> Net-(J15-Pin_22)
- U3 pad 22: Net-(J3-Pin_4) -> Net-(J15-Pin_26)
- U3 pad 23: Net-(J3-Pin_3) -> Net-(J15-Pin_28)
- U3 pad 24: Net-(J3-Pin_2) -> Net-(J15-Pin_30)
- U3 pad 26: unconnected-(U3-XLAT-Pad26) -> /IO40
- U3 pad 28: /VBUS -> /EXT_5V
- U3 pad 3: Net-(J3-Pin_30) -> Net-(J16-Pin_21)
- U3 pad 31: Net-(U1-IO2) -> /IO41
- U3 pad 33: unconnected-(U3-PowerPAD-Pad33) -> /GND
- U3 pad 4: Net-(J3-Pin_28) -> Net-(J16-Pin_25)
- U3 pad 5: Net-(J3-Pin_27) -> Net-(J16-Pin_27)
- U3 pad 6: Net-(J3-Pin_26) -> Net-(J16-Pin_29)
- U3 pad 7: Net-(J3-Pin_24) -> Net-(J16-Pin_33)
- U3 pad 8: Net-(J3-Pin_23) -> Net-(J16-Pin_35)
- U3 pad 9: Net-(J3-Pin_22) -> Net-(J16-Pin_37)
- U4 pad 1: Net-(J4-Pin_32) -> Net-(J16-Pin_46)
- U4 pad 10: Net-(J4-Pin_20) -> Net-(J16-Pin_22)
- U4 pad 11: Net-(J4-Pin_19) -> Net-(J16-Pin_20)
- U4 pad 12: Net-(J4-Pin_18) -> Net-(J16-Pin_18)
- U4 pad 13: Net-(J4-Pin_16) -> Net-(J16-Pin_14)
- U4 pad 14: Net-(J4-Pin_15) -> Net-(J16-Pin_12)
- U4 pad 15: Net-(J4-Pin_14) -> Net-(J16-Pin_10)
- U4 pad 16: Net-(J4-Pin_12) -> Net-(J16-Pin_6)
- U4 pad 17: Net-(J4-Pin_11) -> Net-(J16-Pin_4)
- U4 pad 18: Net-(J4-Pin_10) -> Net-(J16-Pin_2)
- U4 pad 19: Net-(J4-Pin_8) -> Net-(J16-Pin_1)
- U4 pad 2: Net-(J4-Pin_31) -> Net-(J16-Pin_44)
- U4 pad 20: Net-(J4-Pin_7) -> Net-(J16-Pin_3)
- U4 pad 21: Net-(J4-Pin_6) -> Net-(J16-Pin_5)
- U4 pad 22: Net-(J4-Pin_4) -> Net-(J16-Pin_9)
- U4 pad 23: Net-(J4-Pin_3) -> Net-(J16-Pin_11)
- U4 pad 24: Net-(J4-Pin_2) -> Net-(J16-Pin_13)
- U4 pad 26: unconnected-(U4-XLAT-Pad26) -> /IO40
- U4 pad 28: /VBUS -> /EXT_5V
- U4 pad 3: Net-(J4-Pin_30) -> Net-(J16-Pin_42)
- U4 pad 31: Net-(U1-IO2) -> /IO41
- U4 pad 33: unconnected-(U4-PowerPAD-Pad33) -> /GND
- U4 pad 4: Net-(J4-Pin_28) -> Net-(J16-Pin_38)
- U4 pad 5: Net-(J4-Pin_27) -> Net-(J16-Pin_36)
- U4 pad 6: Net-(J4-Pin_26) -> Net-(J16-Pin_34)
- U4 pad 7: Net-(J4-Pin_24) -> Net-(J16-Pin_30)
- U4 pad 8: Net-(J4-Pin_23) -> Net-(J16-Pin_28)
- U4 pad 9: Net-(J4-Pin_22) -> Net-(J16-Pin_26)
- U6 pad 10: /IO3 -> /PD0
- U6 pad 11: /IO46 -> /PD1
- U6 pad 13: /IO11 -> /PD6
- U6 pad 14: /IO10 -> /PD4
- U6 pad 15: /IO9 -> /PD5
- U7 pad 10: /IO3 -> /PD0
- U7 pad 11: /IO46 -> /PD1
- U7 pad 13: /IO11 -> /PD6
- U7 pad 14: /IO10 -> /PD4
- U7 pad 15: /IO12 -> /PD7
- U8 pad 10: unconnected-(U8-PB2-Pad10) -> /MOSI
- U8 pad 11: unconnected-(U8-PB3-Pad11) -> /MISO
- U8 pad 14: /VCC -> /3.3v
- U8 pad 16: unconnected-(U8-XTAL2-Pad16) -> Net-(U8-XTAL2)
- U8 pad 17: unconnected-(U8-XTAL1-Pad17) -> Net-(U8-XTAL1)
- U8 pad 18: unconnected-(U8-PD0-Pad18) -> /PD0
- U8 pad 19: unconnected-(U8-PD1-Pad19) -> /PD1
- U8 pad 2: unconnected-(U8-UVCC-Pad2) -> /VBUS
- U8 pad 20: unconnected-(U8-PD2-Pad20) -> /IO4
- U8 pad 21: unconnected-(U8-PD3-Pad21) -> /IO5
- U8 pad 22: unconnected-(U8-PD5-Pad22) -> /PD5
- U8 pad 24: Net-(U8-AVCC-Pad24) -> /3.3v
- U8 pad 25: unconnected-(U8-PD4-Pad25) -> /PD4
- U8 pad 26: unconnected-(U8-PD6-Pad26) -> /PD6
- U8 pad 27: unconnected-(U8-PD7-Pad27) -> /PD7
- U8 pad 28: unconnected-(U8-PB4-Pad28) -> /CS1
- U8 pad 29: unconnected-(U8-PB5-Pad29) -> /CS2
- U8 pad 3: unconnected-(U8-D--Pad3) -> /D4-
- U8 pad 33: unconnected-(U8-~{HWB}/PE2-Pad33) -> /GND
- U8 pad 34: /VCC -> /3.3v
- U8 pad 4: unconnected-(U8-D+-Pad4) -> /D4+
- U8 pad 42: unconnected-(U8-AREF-Pad42) -> Net-(U8-AREF)
- U8 pad 44: Net-(U8-AVCC-Pad24) -> /3.3v
- U8 pad 5: unconnected-(U8-UGND-Pad5) -> /GND
- U8 pad 6: unconnected-(U8-UCAP-Pad6) -> Net-(U8-UCAP)
- U8 pad 7: unconnected-(U8-VBUS-Pad7) -> /VBUS
- U8 pad 9: unconnected-(U8-PB1-Pad9) -> /SCK
- U9 pad 1: unconnected-(U9-VSS-Pad1) -> /GND
- U9 pad 10: unconnected-(U9-DM1-Pad10) -> /D1-
- U9 pad 11: unconnected-(U9-DP1-Pad11) -> /D1+
- U9 pad 13: unconnected-(U9-VD33-Pad13) -> /3.3v
- U9 pad 14: unconnected-(U9-REXT-Pad14) -> Net-(U9-REXT)
- U9 pad 15: unconnected-(U9-DMU-Pad15) -> /DU-
- U9 pad 16: unconnected-(U9-DPU-Pad16) -> /DU+
- U9 pad 17: unconnected-(U9-~{XRSTJ}-Pad17) -> Net-(U9-~{XRSTJ})
- U9 pad 18: unconnected-(U9-VBUSM-Pad18) -> Net-(U9-VBUSM)
- U9 pad 19: unconnected-(U9-BUSJ-Pad19) -> Net-(U9-BUSJ)
- U9 pad 2: unconnected-(U9-XOUT-Pad2) -> Net-(U9-XOUT)
- U9 pad 20: unconnected-(U9-VDD5-Pad20) -> /VBUS
- U9 pad 26: unconnected-(U9-OVCJ-Pad26) -> /3.3v
- U9 pad 28: unconnected-(U9-VD18-Pad28) -> Net-(U9-VD18)
- U9 pad 3: unconnected-(U9-XIN-Pad3) -> Net-(U9-XIN)
- U9 pad 4: unconnected-(U9-DM4-Pad4) -> /D4-
- U9 pad 5: unconnected-(U9-DP4-Pad5) -> /D4+
- U9 pad 6: unconnected-(U9-DM3-Pad6) -> /D3-
- U9 pad 7: unconnected-(U9-DP3-Pad7) -> /D3+
- U9 pad 8: unconnected-(U9-DM2-Pad8) -> /D2-
- U9 pad 9: unconnected-(U9-DP2-Pad9) -> /D2+
Routing:
- net /VBUS: track 545.8 -> 174.2 mm, vias 6 -> 5
- net /EXT_5V: track 0.00 -> 359.5 mm, vias 0 -> 5
- net Net-(U1-IO2): track 221.7 -> 0.00 mm, vias 5 -> 0
- net /IO38: track 0.00 -> 168.8 mm
- net /IO39: track 0.00 -> 166.9 mm
- net /IO41: track 0.00 -> 156.4 mm, vias 0 -> 4
- net /IO40: track 0.00 -> 151.8 mm, vias 0 -> 6
- net /GND: track 27.6 -> 150.9 mm, vias 13 -> 42
- net /3.3v: track 111.9 -> 230.4 mm, vias 3 -> 10
- net /IO3: track 108.3 -> 0.00 mm, vias 4 -> 0
- net /IO46: track 108.0 -> 0.00 mm, vias 4 -> 0
- net /IO11: track 102.2 -> 0.00 mm, vias 2 -> 0
- net /CS2: track 0.00 -> 100.9 mm
- net /IO10: track 100.6 -> 0.00 mm, vias 2 -> 0
- net /IO12: track 97.4 -> 0.00 mm
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Other:
- board size 252.2 x 44.8 mm -> 146.3 x 55.8 mm

Commit message: board
Parts:
- removed the H2 at (153.7, 79.9)
- removed the H3 at (42.8, 82.7)
- removed the H4 at (92.1, 79.9)
- moved H4 164.1 mm to (153.8, 80.1)
- moved H3 113.8 mm to (91.9, 80.0)
- moved H2 89.4 mm to (42.8, 82.7)
- moved C6 1.14 mm to (83.4, 107.5)
- moved C2 1.14 mm to (83.4, 105.6)
- moved J16 0.07 mm to (98.3, 73.3)
Connections:
- U3 pad 1: Net-(J16-Pin_17) -> Net-(J16-Pin_18)
- U3 pad 10: Net-(J16-Pin_41) -> Net-(J16-Pin_42)
- U3 pad 11: Net-(J16-Pin_43) -> Net-(J16-Pin_44)
- U3 pad 12: Net-(J16-Pin_45) -> Net-(J16-Pin_46)
- U3 pad 2: Net-(J16-Pin_19) -> Net-(J16-Pin_20)
- U3 pad 3: Net-(J16-Pin_21) -> Net-(J16-Pin_22)
- U3 pad 4: Net-(J16-Pin_25) -> Net-(J16-Pin_26)
- U3 pad 5: Net-(J16-Pin_27) -> Net-(J16-Pin_28)
- U3 pad 6: Net-(J16-Pin_29) -> Net-(J16-Pin_30)
- U3 pad 7: Net-(J16-Pin_33) -> Net-(J16-Pin_34)
- U3 pad 8: Net-(J16-Pin_35) -> Net-(J16-Pin_36)
- U3 pad 9: Net-(J16-Pin_37) -> Net-(J16-Pin_38)
- U4 pad 1: Net-(J16-Pin_46) -> Net-(J16-Pin_45)
- U4 pad 10: Net-(J16-Pin_22) -> Net-(J16-Pin_21)
- U4 pad 11: Net-(J16-Pin_20) -> Net-(J16-Pin_19)
- U4 pad 12: Net-(J16-Pin_18) -> Net-(J16-Pin_17)
- U4 pad 13: Net-(J16-Pin_14) -> Net-(J16-Pin_13)
- U4 pad 14: Net-(J16-Pin_12) -> Net-(J16-Pin_11)
- U4 pad 15: Net-(J16-Pin_10) -> Net-(J16-Pin_9)
- U4 pad 16: Net-(J16-Pin_6) -> Net-(J16-Pin_5)
- U4 pad 17: Net-(J16-Pin_4) -> Net-(J16-Pin_3)
- U4 pad 18: Net-(J16-Pin_2) -> Net-(J16-Pin_1)
- U4 pad 19: Net-(J16-Pin_1) -> Net-(J16-Pin_2)
- U4 pad 2: Net-(J16-Pin_44) -> Net-(J16-Pin_43)
- U4 pad 20: Net-(J16-Pin_3) -> Net-(J16-Pin_4)
- U4 pad 21: Net-(J16-Pin_5) -> Net-(J16-Pin_6)
- U4 pad 22: Net-(J16-Pin_9) -> Net-(J16-Pin_10)
- U4 pad 23: Net-(J16-Pin_11) -> Net-(J16-Pin_12)
- U4 pad 24: Net-(J16-Pin_13) -> Net-(J16-Pin_14)
- U4 pad 3: Net-(J16-Pin_42) -> Net-(J16-Pin_41)
- U4 pad 4: Net-(J16-Pin_38) -> Net-(J16-Pin_37)
- U4 pad 5: Net-(J16-Pin_36) -> Net-(J16-Pin_35)
- U4 pad 6: Net-(J16-Pin_34) -> Net-(J16-Pin_33)
- U4 pad 7: Net-(J16-Pin_30) -> Net-(J16-Pin_29)
- U4 pad 8: Net-(J16-Pin_28) -> Net-(J16-Pin_27)
- U4 pad 9: Net-(J16-Pin_26) -> Net-(J16-Pin_25)
Routing:
- net Net-(J16-Pin_13): track 59.1 -> 15.4 mm
- net Net-(J16-Pin_45): track 70.7 -> 28.1 mm
- net Net-(J16-Pin_43): track 67.3 -> 25.4 mm
- net Net-(J16-Pin_41): track 63.9 -> 22.6 mm
- net Net-(J16-Pin_14): track 17.4 -> 58.1 mm
- net Net-(J16-Pin_37): track 57.4 -> 17.4 mm
- net Net-(J16-Pin_35): track 53.9 -> 14.6 mm
- net Net-(J16-Pin_33): track 51.2 -> 11.9 mm
- net Net-(J16-Pin_29): track 45.9 -> 7.27 mm
- net Net-(J16-Pin_27): track 43.1 -> 5.46 mm
- net Net-(J16-Pin_11): track 54.9 -> 17.4 mm
- net Net-(J16-Pin_25): track 40.1 -> 4.00 mm
- net Net-(J16-Pin_46): track 30.8 -> 66.3 mm
- net Net-(J16-Pin_44): track 27.6 -> 62.9 mm
- net Net-(J16-Pin_42): track 24.7 -> 59.5 mm
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
Commit message: duplicated PCB
Parts:
- removed C10, C11, C12, C13, C14, C3, C4: 22pf, Capacitor_SMD:C_0603_1608Metric_Pad1.08x0.95mm_HandSolder
- removed Y1: Crystal_GND24, Crystal:Crystal_SMD_2520-4Pin_2.5x2.0mm
- added C15: 100nf, Capacitor_SMD:C_0603_1608Metric_Pad1.08x0.95mm_HandSolder, F.Cu at (38.3, 97.6)
- added C16: 2.2uf, Capacitor_SMD:C_0603_1608Metric_Pad1.08x0.95mm_HandSolder, F.Cu at (36.5, 97.6)
- added C17: 100nf, Capacitor_SMD:C_0603_1608Metric_Pad1.08x0.95mm_HandSolder, F.Cu at (36.6, 107.7)
- added C18: 100nf, Capacitor_SMD:C_0603_1608Metric_Pad1.08x0.95mm_HandSolder, F.Cu at (42.1, 112.0)
- added C19: 100nf, Capacitor_SMD:C_0603_1608Metric_Pad1.08x0.95mm_HandSolder, F.Cu at (47.1, 107.6)
- added C20: 100nf, Capacitor_SMD:C_0603_1608Metric_Pad1.08x0.95mm_HandSolder, F.Cu at (36.6, 104.2)
- added C21: 100nf, Capacitor_SMD:C_0603_1608Metric_Pad1.08x0.95mm_HandSolder, F.Cu at (40.0, 97.6)
- added C22: 100nf, Capacitor_SMD:C_0603_1608Metric_Pad1.08x0.95mm_HandSolder, F.Cu at (47.1, 104.1)
- added C23: 100nf, Capacitor_SMD:C_0603_1608Metric_Pad1.08x0.95mm_HandSolder, F.Cu at (45.0, 112.0)
- added C24: 100nf, Capacitor_SMD:C_0603_1608Metric_Pad1.08x0.95mm_HandSolder, F.Cu at (34.8, 112.6)
- added R10: 5.1k, Resistor_SMD:R_0603_1608Metric_Pad0.98x0.95mm_HandSolder, F.Cu at (40.3, 112.0)
- added R11: 27, Resistor_SMD:R_0603_1608Metric_Pad0.98x0.95mm_HandSolder, F.Cu at (44.2, 99.9)
- added R12: 27, Resistor_SMD:R_0603_1608Metric_Pad0.98x0.95mm_HandSolder, F.Cu at (42.6, 99.9)
- added Y3: Crystal_GND24, Crystal:Crystal_SMD_2520-4Pin_2.5x2.0mm, F.Cu at (37.5, 112.6)
- U1: value ESP32-S3-WROOM-1 -> RP2040; footprint RF_Module:ESP32-S3-WROOM-1 -> Package_DFN_QFN:QFN-56-1EP_7x7mm_P0.4mm_EP3.2x3.2mm
- U8: value ATmega32U4-M -> W25Q16JVSS; footprint Package_DFN_QFN:QFN-44-1EP_7x7mm_P0.5mm_EP5.2x5.2mm -> Package_SO:SOIC-8_5.3x5.3mm_P1.27mm
- moved U8 39.4 mm to (32.9, 105.9), turned to -90 degrees
- moved U1 4.02 mm to (41.9, 105.8), turned to 0 degrees
Connections:
- J2 pad 3: /IO39 -> unconnected-(J2-Pin_3-Pad3)
- U1 pad 1: /GND -> /3.3v
- U1 pad 10: unconnected-(U1-IO17-Pad10) -> /3.3v
- U1 pad 12: /IO8 -> unconnected-(U1-GPIO9-Pad12)
- U1 pad 13: /D1- -> unconnected-(U1-GPIO10-Pad13)
- U1 pad 14: /D1+ -> unconnected-(U1-GPIO11-Pad14)
- U1 pad 15: /IO3 -> unconnected-(U1-GPIO12-Pad15)
- U1 pad 16: /IO46 -> unconnected-(U1-GPIO13-Pad16)
- U1 pad 17: /IO9 -> unconnected-(U1-GPIO14-Pad17)
- U1 pad 18: /IO10 -> unconnected-(U1-GPIO15-Pad18)
- U1 pad 19: /IO11 -> unconnected-(U1-TESTEN-Pad19)
- U1 pad 2: /3.3v -> unconnected-(U1-GPIO0-Pad2)
- U1 pad 20: /IO12 -> /XIN
- U1 pad 21: /IO13 -> /XOUT
- U1 pad 22: /IO14 -> /3.3v
- U1 pad 23: unconnected-(U1-IO21-Pad23) -> Net-(U1-DVDD-Pad23)
- U1 pad 31: /IO38 -> unconnected-(U1-GPIO20-Pad31)
- U1 pad 32: /IO39 -> unconnected-(U1-GPIO21-Pad32)
- U1 pad 33: /IO40 -> /3.3v
- U1 pad 34: /IO41 -> unconnected-(U1-GPIO22-Pad34)
- U1 pad 35: /IO42 -> unconnected-(U1-GPIO23-Pad35)
- U1 pad 36: /RXD0 -> unconnected-(U1-GPIO24-Pad36)
- U1 pad 37: /TXD0 -> unconnected-(U1-GPIO25-Pad37)
- U1 pad 4: /IO4 -> unconnected-(U1-GPIO2-Pad4)
- U1 pad 40: /GND -> unconnected-(U1-GPIO28/ADC2-Pad40)
- U1 pad 41: /GND -> unconnected-(U1-GPIO29/ADC3-Pad41)
- U1 pad 5: /IO5 -> unconnected-(U1-GPIO3-Pad5)
- U1 pad 6: /IO6 -> unconnected-(U1-GPIO4-Pad6)
- U1 pad 7: /IO7 -> unconnected-(U1-GPIO5-Pad7)
- U1 pad 8: /IO15 -> unconnected-(U1-GPIO6-Pad8)
- U1 pad 9: /IO16 -> unconnected-(U1-GPIO7-Pad9)
- U8 pad 1: unconnected-(U8-PE6-Pad1) -> /QSPI_SS
- U8 pad 2: /VBUS -> /QSPI_SD1
- U8 pad 3: /D4- -> /QSPI_SD2
- U8 pad 4: /D4+ -> /GND
- U8 pad 5: /GND -> /QSPI_SD0
- U8 pad 6: Net-(U8-UCAP) -> /QSPI_SCLK
- U8 pad 7: /VBUS -> /QSPI_SD3
- U8 pad 8: unconnected-(U8-PB0-Pad8) -> /3.3v
Routing:
- net /IO38: track 168.8 -> 0.00 mm
- net /IO39: track 166.9 -> 0.00 mm
- net /CS2: track 100.9 -> 0.00 mm
- net /CS1: track 96.2 -> 0.00 mm
- net /PD7: track 94.1 -> 0.00 mm
- net /IO5: track 83.0 -> 0.00 mm, vias 2 -> 0
- net /IO4: track 78.7 -> 0.00 mm, vias 2 -> 0
- net /GND: track 132.5 -> 71.6 mm, vias 42 -> 36
- net /IO42: track 64.7 -> 7.56 mm
- net /IO41: track 156.8 -> 101.3 mm
- net /IO40: track 150.5 -> 96.4 mm
- net /PD6: track 96.2 -> 59.9 mm
- net /PD4: track 93.7 -> 59.0 mm
- net /PD5: track 30.3 -> 0.00 mm
- net /QSPI_SD3: track 0.00 -> 28.8 mm
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