File: PCB/arcade/arcade.kicad_pcb (KiCad board)
At the start: 4 copper layers, 146.3 x 63 mm, 45 parts, among them J1 USB_C_Receptacle_USB2.0_16P, J15 Conn_02x24_Odd_Even, J16 Conn_02x24_Odd_Even, J2 Conn_02x03_Odd_Even, J3 Conn_02x06_Odd_Even, J4 Screw_Terminal_01x02, J5 Screw_Terminal_01x12, J6 Screw_Terminal_01x08, J7 Screw_Terminal_01x12, J8 Conn_01x02_Pin, J9 Conn_01x06_Pin, U1 RP2040, U2 TLC5947RHB, U3 TLC5947RHB, U4 TLC5947RHB, U5 ME6211C33M5, U6 CD74HC4067M, U7 CD74HC4067M, U8 W25Q16JVSS, U9 TS3USB221ARSERG4, Y3 Crystal_GND24

Commit message: board changes
Parts:
- added J10: Conn_02x06_Odd_Even, Connector_PinHeader_2.54mm:PinHeader_2x06_P2.54mm_Horizontal, F.Cu at (209.3, 78.7)
- added J11: USB_C_Receptacle_USB2.0_16P, Connector_USB:USB_C_Receptacle_GCT_USB4110, F.Cu at (172.5, 111.6)
- added J12: USB_C_Receptacle_USB2.0_16P, Connector_USB:USB_C_Receptacle_GCT_USB4110, F.Cu at (158.0, 111.6)
- added J13: HDMI_A_1.4, Connector_Video:HDMI_A_Amphenol_10029449-x01xLF_Horizontal, F.Cu at (118.7, 111.6)
- added J14: USB_C_Receptacle, Connector_USB:USB_C_Receptacle_Amphenol_12401548E4-2A, F.Cu at (134.0, 111.0)
- added J17: USB_C_Receptacle, Connector_USB:USB_C_Receptacle_Amphenol_12401548E4-2A, F.Cu at (145.0, 111.0)
- added U10: TCA9548AMRGER, Package_DFN_QFN:Texas_RGE0024C_VQFN-24-1EP_4x4mm_P0.5mm_EP2.1x2.1mm, F.Cu at (81.9, 106.2)
- moved H1 148.5 mm to (217.0, 110.0)
- moved Module1 120.2 mm to (201.7, 70.5), turned to -90 degrees
- moved J3 119.6 mm to (36.0, 92.1), turned to 180 degrees
- moved H3 92.0 mm to (69.0, 111.0)
- moved U7 78.3 mm to (66.2, 93.4), turned to -90 degrees
- moved J7 72.0 mm to (72.3, 83.0), turned to 180 degrees
- moved H4 68.8 mm to (219.0, 56.0)
- moved J5 53.7 mm to (127.5, 83.0), turned to 180 degrees
- moved J6 36.1 mm to (94.8, 83.0), turned to 180 degrees
- moved C1 27.0 mm to (49.5, 91.3)
- moved C2 27.0 mm to (50.5, 96.4)
- moved C6 27.0 mm to (50.5, 98.3)
- moved U5 27.0 mm to (49.3, 93.8)
- moved J4 19.2 mm to (166.5, 57.8), turned to 180 degrees
- moved U6 18.1 mm to (113.0, 93.4), turned to -90 degrees
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Routing:
- net /MISO: track 74.8 -> 0.00 mm, vias 2 -> 0
- net /MOSI: track 74.1 -> 0.00 mm, vias 2 -> 0
- net /SCK: track 73.3 -> 0.00 mm, vias 2 -> 0
- net /3.3v: track 177.0 -> 138.6 mm
- net /EXT_5V: track 365.7 -> 343.3 mm
- net /GND: track 50.1 -> 47.6 mm, vias 33 -> 31
- net /IO40: track 97.9 -> 99.1 mm
Other:
- board size 146.3 x 63 mm -> 200.1 x 63 mm

Commit message: analog working
Parts:
- removed J14, J17: USB_C_Receptacle, Connector_USB:USB_C_Receptacle_Amphenol_12401548E4-2A
- J10: value Conn_02x06_Odd_Even -> USB3_A_Stacked; footprint Connector_PinHeader_2.54mm:PinHeader_2x06_P2.54mm_Horizontal -> Connector_USB:USB3_A_Molex_48406-0001_Horizontal_Stacked
- J11: value USB_C_Receptacle_USB2.0_16P -> USB_A_Stacked; footprint Connector_USB:USB_C_Receptacle_GCT_USB4110 -> Connector_USB:USB_A_CUI_UJ2-ADH-TH_Horizontal_Stacked
- J12: value USB_C_Receptacle_USB2.0_16P -> RJ45_RB1-125B8G1A; footprint Connector_USB:USB_C_Receptacle_GCT_USB4110 -> Connector_RJ:RJ45_UDE_RB1-125B8G1A
- moved J13 81.3 mm to (200.0, 112.0)
- moved J10 41.5 mm to (177.5, 105.3)
- moved J2 26.1 mm to (158.9, 43.5)
- moved J12 26.1 mm to (136.3, 97.1)
- moved J4 17.7 mm to (178.5, 44.8)
- moved Module1 16.9 mm to (216.0, 61.5)
- moved J11 16.0 mm to (158.5, 103.9), turned to 90 degrees
- moved J3 0.46 mm to (36.0, 91.6)
Connections:
- J10 pad 1: /CS1 -> unconnected-(J10A-VBUS1-Pad1)
- J10 pad 10: /3.3v -> (no net)
- J10 pad 11: /GND -> (no net)
- J10 pad 12: /GND -> (no net)
- J10 pad 2: /CS2 -> unconnected-(J10A-D1--Pad2)
- J10 pad 3: /MISO -> unconnected-(J10A-D1+-Pad3)
- J10 pad 4: /MISO -> unconnected-(J10A-GND1-Pad4)
- J10 pad 5: /MOSI -> unconnected-(J10A-SSRX1--Pad5)
- J10 pad 6: /MOSI -> unconnected-(J10A-SSRX1+-Pad6)
- J10 pad 7: /SCK -> unconnected-(J10A-DRAIN1-Pad7)
- J10 pad 8: /SCK -> unconnected-(J10A-SSTX1--Pad8)
- J10 pad 9: /3.3v -> unconnected-(J10A-SSTX1+-Pad9)
- J11 pad SH: (no net) -> unconnected-(J11-Shield-PadSH)
- J12 pad SH: (no net) -> unconnected-(J12-PadSH)
