File: PCB/arcade/arcade.kicad_sch (KiCad schematic)
At the start: 17 parts, among them J1 USB_C_Receptacle_USB2.0_16P, J2 Conn_01x32_Pin, J3 Conn_01x32_Pin, J4 Conn_01x32_Pin, J5 Screw_Terminal_01x12, J6 Screw_Terminal_01x12, J7 Screw_Terminal_01x04, U1 ESP32-S3-WROOM-1, U2 TLC5947RHB, U3 TLC5947RHB, U4 TLC5947RHB, U5 ME6211C33M5

Commit message: pcb
Parts:
- removed J6: Screw_Terminal_01x12, TerminalBlock_Phoenix:TerminalBlock_Phoenix_MPT-0,5-12-2.54_1x12_P2.54mm_Horizontal, symbol Connector:Screw_Terminal_01x12
- removed J7: Screw_Terminal_01x04, TerminalBlock_Phoenix:TerminalBlock_Phoenix_MPT-0,5-4-2.54_1x04_P2.54mm_Horizontal, symbol Connector:Screw_Terminal_01x04
- added C3, C4: 22pf, Capacitor_SMD:C_0603_1608Metric_Pad1.08x0.95mm_HandSolder, symbol Device:C
- added C5, C7: .01uf, Capacitor_SMD:C_0603_1608Metric_Pad1.08x0.95mm_HandSolder, symbol Device:C
- added FB2: FerriteBead, Inductor_SMD:L_0603_1608Metric, symbol Device:FerriteBead
- added J6: Screw_Terminal_01x08, TerminalBlock_Phoenix:TerminalBlock_Phoenix_MPT-0,5-8-2.54_1x08_P2.54mm_Horizontal, symbol Connector:Screw_Terminal_01x08
- added J7: Screw_Terminal_01x12, TerminalBlock_Phoenix:TerminalBlock_Phoenix_MPT-0,5-12-2.54_1x12_P2.54mm_Horizontal, symbol Connector:Screw_Terminal_01x12
- added R1, R2: 22, Resistor_SMD:R_0603_1608Metric_Pad0.98x0.95mm_HandSolder, symbol Device:R_US
- added R3, R6: 10k, Resistor_SMD:R_0603_1608Metric_Pad0.98x0.95mm_HandSolder, symbol Device:R_US
- added U6, U7: CD74HC4067M, Package_SO:SSOP-24_5.3x8.2mm_P0.65mm, symbol 74xx:CD74HC4067M
- added U8: MAX3421EEHJ+T, max3421:21-0110-C_90-0149-32L_MXM, symbol max:MAX3421EEHJ+T
- added Y1: Crystal_GND24, Crystal:Crystal_SMD_2520-4Pin_2.5x2.0mm, symbol Device:Crystal_GND24
Connections:
- net 3.3v: now also R3.2, R6.1, U8.2 (VL), U8.23 (VCC)
- net VBUS: now reaches C1.1, J1.A4 (VBUS), J1.A9 (VBUS), J1.B4 (VBUS), J1.B9 (VBUS), J2.1 (Pin_1), J2.13 (Pin_13), J2.17 (Pin_17), J2.21 (Pin_21), J2.25 (Pin_25), J2.29 (Pin_29), J2.5 (Pin_5), J2.9 (Pin_9), J3.1 (Pin_1), J3.13 (Pin_13), J3.17 (Pin_17), J3.21 (Pin_21), J3.25 (Pin_25), J3.29 (Pin_29), J3.5 (Pin_5), J3.9 (Pin_9), J4.1 (Pin_1), J4.13 (Pin_13), J4.17 (Pin_17), J4.21 (Pin_21), J4.25 (Pin_25), J4.29 (Pin_29), J4.5 (Pin_5), J4.9 (Pin_9), U2.28 (VCC), U3.28 (VCC), U4.28 (VCC), U5.1 (V_{IN}), U5.3 (CE)
- net VBUS: now also FB2.2
- net at C1.2, C2.2, C6.2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: now also R4.2, R5.2
- net IO10: now reaches U1.18 (IO10)
- net IO10: now also U6.14 (S2), U7.14 (S2), U8.14 (*SS)
- net IO11: now reaches U1.19 (IO11)
- net IO11: now also U6.13 (S3), U7.13 (S3), U8.16 (MOSI)
- net IO12: now reaches U1.20 (IO12)
- net IO12: now also U7.15 (~{E}), U8.13 (SCLK)
- net IO13: now reaches U1.21 (IO13)
- net IO13: now also U8.15 (MISO)
- net IO14: now reaches U1.22 (IO14)
- net at J5.7 (Pin_7): now also U6.4 (I5); no longer U1.10 (IO17)
- net at J5.8 (Pin_8): now also U6.5 (I4); no longer U1.11 (IO18)
- net at J5.9 (Pin_9): now also U6.6 (I3); no longer U1.12 (IO8)
- net at J5.10 (Pin_10): now also U6.7 (I2); no longer U1.15 (IO3)
- net at J5.11 (Pin_11): now also U6.8 (I1); no longer U1.16 (IO46)
- net at J5.12 (Pin_12): now also U6.9 (I0); no longer U1.17 (IO9)
- net at J5.1 (Pin_1): now also U6.20 (I11); no longer U1.4 (IO4)
- net at J5.2 (Pin_2): now also U6.21 (I10); no longer U1.5 (IO5)
- net at J5.3 (Pin_3): now also U6.22 (I9); no longer U1.6 (IO6)
- net at J5.4 (Pin_4): now also U6.23 (I8); no longer U1.7 (IO7)
- net at J5.5 (Pin_5): now also U6.2 (I7); no longer U1.8 (IO15)
- net at J5.6 (Pin_6): now also U6.3 (I6); no longer U1.9 (IO16)
- new net: J7.12 (Pin_12), U7.16 (I15)
- new net: J7.11 (Pin_11), U7.17 (I14)
- new net: J7.10 (Pin_10), U7.18 (I13)
- new net: J7.9 (Pin_9), U7.19 (I12)
- new net: J7.4 (Pin_4), U7.2 (I7)
- new net: J7.8 (Pin_8), U7.20 (I11)
- new net: J7.7 (Pin_7), U7.21 (I10)
- new net: J7.6 (Pin_6), U7.22 (I9)
- new net: J7.5 (Pin_5), U7.23 (I8)
- new net: J7.3 (Pin_3), U7.3 (I6)
- new net: J7.2 (Pin_2), U7.4 (I5)
- new net: J7.1 (Pin_1), U7.5 (I4)
- new net: J6.8 (Pin_8), U7.6 (I3)
- new net: J6.7 (Pin_7), U7.7 (I2)
- new net: J6.6 (Pin_6), U7.8 (I1)
- new net: J6.5 (Pin_5), U7.9 (I0)
- new net: R3.1, U8.18 (INT)
- new net: C3.1, C4.1, C5.2
- new net: C3.2, U8.25 (XO), Y1.3
- new net: C5.1, FB2.1
- new net: R6.2, U8.12 (*RES)
- new net: C7.2, U8.19 (GND), U8.3 (GND), Y1.2, Y1.4
- new net: R1.2, U8.20 (D-)
- new net: R2.2, U8.21 (D+)
- new net: C7.1, U8.22 (VBCOMP)
- new net: C4.2, U8.24 (XI), Y1.1
- new net: J6.4 (Pin_4), U6.16 (I15)
- new net: J6.3 (Pin_3), U6.17 (I14)
- new net: J6.2 (Pin_2), U6.18 (I13)
- new net: J6.1 (Pin_1), U6.19 (I12)
- new net IO15: U1.8 (IO15)
- new net IO16: U1.9 (IO16)
- new net IO3: U1.15 (IO3), U6.10 (S0), U7.10 (S0)
- new net IO46: U1.16 (IO46), U6.11 (S1), U7.11 (S1)
- new net IO9: U1.17 (IO9), U6.15 (~{E})
Other:
- moved on the sheet: J5

Commit message: stopping point on PCB
Parts:
- removed C3, C4: 22pf, Capacitor_SMD:C_0603_1608Metric_Pad1.08x0.95mm_HandSolder, symbol Device:C
- removed C5, C7: .01uf, Capacitor_SMD:C_0603_1608Metric_Pad1.08x0.95mm_HandSolder, symbol Device:C
- removed FB2: FerriteBead, Inductor_SMD:L_0603_1608Metric, symbol Device:FerriteBead
- removed R1, R2: 22, Resistor_SMD:R_0603_1608Metric_Pad0.98x0.95mm_HandSolder, symbol Device:R_US
- removed R3, R6: 10k, Resistor_SMD:R_0603_1608Metric_Pad0.98x0.95mm_HandSolder, symbol Device:R_US
- removed U8: MAX3421EEHJ+T, max3421:21-0110-C_90-0149-32L_MXM, symbol max:MAX3421EEHJ+T
- removed Y1: Crystal_GND24, Crystal:Crystal_SMD_2520-4Pin_2.5x2.0mm, symbol Device:Crystal_GND24
- added J10, J11: USB_A, Connector_USB:USB_A_Molex_67643_Horizontal, symbol Connector:USB_A
- added J12, J13: Conn_01x06_Pin, Connector_PinHeader_2.54mm:PinHeader_1x06_P2.54mm_Horizontal, symbol Connector:Conn_01x06_Pin
- added J14: Conn_01x04_Pin, Connector_PinHeader_2.54mm:PinHeader_1x04_P2.54mm_Vertical, symbol Connector:Conn_01x04_Pin
- added J8, J9: Conn_01x03_Pin, Connector_PinHeader_2.54mm:PinHeader_1x03_P2.54mm_Horizontal, symbol Connector:Conn_01x03_Pin
- added U8: ATmega32U4-M, Package_DFN_QFN:QFN-44-1EP_7x7mm_P0.5mm_EP5.2x5.2mm, symbol MCU_Microchip_ATmega:ATmega32U4-M
- added U9: FE1.1s, Package_SO:SSOP-28_3.9x9.9mm_P0.635mm, symbol Interface_USB:FE1.1s
Connections:
- net 3.3v: now also U6.24 (VCC), U7.24 (VCC)
- net GND: now reaches U2.29 (GND), U3.29 (GND), U4.29 (GND)
- net GND: now also C1.2, C2.2, C6.2, J1.A1 (GND), J1.A12 (GND), J1.B1 (GND), J1.B12 (GND), J1.S1 (SHIELD), R4.2, R5.2, U1.1 (GND), U1.40 (GND), U1.41 (GND), U5.2 (V_{SS}), U6.12 (GND), U7.12 (GND), U8.15 (GND), U8.23 (GND), U8.35 (GND), U8.43 (GND), U8.45 (GND)
- new net: U8.24 (AVCC), U8.44 (AVCC)
- new net VCC: U8.14 (VCC), U8.34 (VCC)

Commit message: board
Parts:
- removed J12, J13: Conn_01x06_Pin, Connector_PinHeader_2.54mm:PinHeader_1x06_P2.54mm_Horizontal, symbol Connector:Conn_01x06_Pin
- removed J14: Conn_01x04_Pin, Connector_PinHeader_2.54mm:PinHeader_1x04_P2.54mm_Vertical, symbol Connector:Conn_01x04_Pin
- removed J2, J3, J4: Conn_01x32_Pin, Connector_PinHeader_2.54mm:PinHeader_1x32_P2.54mm_Horizontal, symbol Connector:Conn_01x32_Pin
- removed J8, J9: Conn_01x03_Pin, Connector_PinHeader_2.54mm:PinHeader_1x03_P2.54mm_Horizontal, symbol Connector:Conn_01x03_Pin
- added C10, C11, C12, C13, C14, C3, C4, C5, C7, C8, C9: 22pf, Capacitor_SMD:C_0603_1608Metric_Pad1.08x0.95mm_HandSolder, symbol Device:C
- added D1: SK6812MINI-E, LED_SMD:LED_SK6812MINI_PLCC4_3.5x3.5mm_P1.75mm, symbol LED:SK6812MINI-E
- added H1, H2, H3, H4: MountingHole, MountingHole:MountingHole_2.5mm_Pad_TopBottom, symbol Mechanical:MountingHole
- added J15, J16: Conn_02x24_Odd_Even, Connector_PinHeader_2.54mm:PinHeader_2x24_P2.54mm_Horizontal, symbol Connector_Generic:Conn_02x24_Odd_Even
- added J2: Conn_02x03_Odd_Even, Connector_PinHeader_2.54mm:PinHeader_2x03_P2.54mm_Horizontal, symbol Connector_Generic:Conn_02x03_Odd_Even
- added J3: Conn_02x06_Odd_Even, Connector_PinHeader_2.54mm:PinHeader_2x06_P2.54mm_Horizontal, symbol Connector_Generic:Conn_02x06_Odd_Even
- added J4: Screw_Terminal_01x02, TerminalBlock_Phoenix:TerminalBlock_Phoenix_MKDS-3-2-5.08_1x02_P5.08mm_Horizontal, symbol Connector:Screw_Terminal_01x02
- added J8: Conn_01x02_Pin, Connector_PinHeader_2.54mm:PinHeader_1x02_P2.54mm_Vertical, symbol Connector:Conn_01x02_Pin
- added J9: Conn_01x06_Pin, Connector_PinHeader_2.54mm:PinHeader_1x06_P2.54mm_Vertical, symbol Connector:Conn_01x06_Pin
- added R6, R7, R8, R9: 5.1k, Resistor_SMD:R_0603_1608Metric_Pad0.98x0.95mm_HandSolder, symbol Device:R_US
- added Y1, Y2: Crystal_GND24, Crystal:Crystal_SMD_2520-4Pin_2.5x2.0mm, symbol Device:Crystal_GND24
Connections:
- net VCC is gone; now on net 3.3v: U8.14 (VCC), U8.34 (VCC)
- net 3.3v: now also U8.24 (AVCC), U8.44 (AVCC), U9.13 (VD33), U9.26 (OVCJ), C12.1, C13.1, C7.1, J3.10 (Pin_10), J3.9 (Pin_9), R7.2, R8.2, R9.2
- net GND: now also J10.4 (GND), J10.SH (Shield), J11.4 (GND), J11.SH (Shield), U2.33 (PowerPAD), U3.33 (PowerPAD), U4.33 (PowerPAD), U8.33 (~{HWB}/PE2), U8.5 (UGND), U9.1 (VSS), C10.2, C11.2, C12.2, C13.2, C14.2, C3.1, C4.1, C5.2, C7.2, C8.2, C9.2, D1.3 (VDD), J2.1 (Pin_1), J2.2 (Pin_2), J3.11 (Pin_11), J3.12 (Pin_12), J4.1 (Pin_1), J9.6 (Pin_6), R6.1, Y1.2, Y1.4, Y2.2, Y2.4
- net IO10: no longer U6.14 (S2), U7.14 (S2)
- net IO11: no longer U6.13 (S3), U7.13 (S3)
- net IO12: no longer U7.15 (~{E})
- net IO14: now also D1.2 (DIN)
- net IO3: no longer U6.10 (S0), U7.10 (S0)
- net IO46: no longer U6.11 (S1), U7.11 (S1)
- net IO9: no longer U6.15 (~{E})
- net VBUS: now also J10.1 (VBUS), J11.1 (VBUS), U8.2 (UVCC), U8.7 (VBUS), U9.20 (VDD5), C14.1, C5.1, D1.1 (VSS), J8.2 (Pin_2), J9.4 (Pin_4); no longer U2.28 (VCC), U3.28 (VCC), U4.28 (VCC)
- net at U3.1 (OUT0): now also J16.17 (Pin_17)
- net at U3.10 (OUT9): now also J16.41 (Pin_41)
- net at U3.11 (OUT10): now also J16.43 (Pin_43)
- net at U3.12 (OUT11): now also J16.45 (Pin_45)
- net at U3.13 (OUT12): now also J15.2 (Pin_2)
- net at U3.14 (OUT13): now also J15.4 (Pin_4)
- net at U3.15 (OUT14): now also J15.6 (Pin_6)
- net at U3.16 (OUT15): now also J15.10 (Pin_10)
- net at U3.17 (OUT16): now also J15.12 (Pin_12)
- net at U3.18 (OUT17): now also J15.14 (Pin_14)
- net at U3.19 (OUT18): now also J15.18 (Pin_18)
- net at U3.2 (OUT1): now also J16.19 (Pin_19)
- net at U3.20 (OUT19): now also J15.20 (Pin_20)
- net at U3.21 (OUT20): now also J15.22 (Pin_22)
- net at U3.22 (OUT21): now also J15.26 (Pin_26)
- net at U3.23 (OUT22): now also J15.28 (Pin_28)
- net at U3.24 (OUT23): now also J15.30 (Pin_30)
- net IO40: now reaches U3.26 (XLAT)
- net IO40: now also U1.33 (IO40), U2.26 (XLAT), U4.26 (XLAT)
- net at U3.3 (OUT2): now also J16.21 (Pin_21)
- net IO41: now reaches U2.31 (SCLK), U3.31 (SCLK), U4.31 (SCLK)
- net IO41: now also U1.34 (IO41); no longer U1.38 (IO2)
- net at U3.4 (OUT3): now also J16.25 (Pin_25)
- net at U3.5 (OUT4): now also J16.27 (Pin_27)
- net at U3.6 (OUT5): now also J16.29 (Pin_29)
- net at U3.7 (OUT6): now also J16.33 (Pin_33)
- net at U3.8 (OUT7): now also J16.35 (Pin_35)
- net at U3.9 (OUT8): now also J16.37 (Pin_37)
- net at U2.18 (OUT17): now also J15.17 (Pin_17)
- net at U2.17 (OUT16): now also J15.19 (Pin_19)
- net at U2.16 (OUT15): now also J15.21 (Pin_21)
- net at U2.15 (OUT14): now also J15.25 (Pin_25)
- net at U2.14 (OUT13): now also J15.27 (Pin_27)
- net at U2.13 (OUT12): now also J15.29 (Pin_29)
- net at U2.12 (OUT11): now also J15.33 (Pin_33)
- net at U2.11 (OUT10): now also J15.35 (Pin_35)
- net at U2.24 (OUT23): now also J15.1 (Pin_1)
- net at U2.10 (OUT9): now also J15.37 (Pin_37)
- net at U2.9 (OUT8): now also J15.41 (Pin_41)
- net at U2.8 (OUT7): now also J15.43 (Pin_43)
- net at U2.7 (OUT6): now also J15.45 (Pin_45)
- net at U2.6 (OUT5): now also J15.46 (Pin_46)
- net at U2.5 (OUT4): now also J15.44 (Pin_44)
- net at U2.4 (OUT3): now also J15.42 (Pin_42)
- net at U2.23 (OUT22): now also J15.3 (Pin_3)
- net at U2.3 (OUT2): now also J15.38 (Pin_38)
- net at U2.2 (OUT1): now also J15.36 (Pin_36)
- net at U2.1 (OUT0): now also J15.34 (Pin_34)
- net at U2.22 (OUT21): now also J15.5 (Pin_5)
- net at U2.21 (OUT20): now also J15.9 (Pin_9)
- net at U2.20 (OUT19): now also J15.11 (Pin_11)
- net at U2.19 (OUT18): now also J15.13 (Pin_13)
- net D1-: now reaches U9.10 (DM1)
- net D1-: now also U1.13 (USB_D-)
- net D1+: now reaches U9.11 (DP1)
- net D1+: now also U1.14 (USB_D+)
- net at U9.14 (REXT): now also R6.2
- net DU-: now reaches U9.15 (DMU)
- net DU-: now also J1.A7 (D-), J1.B7 (D-)
- net DU+: now reaches U9.16 (DPU)
- net DU+: now also J1.A6 (D+), J1.B6 (D+)
- net at U9.17 (~{XRSTJ}): now also R8.1
- net at U9.18 (VBUSM): now also R7.1
- net at U9.19 (BUSJ): now also R9.1
- net at U9.2 (XOUT): now also Y2.1
- net at U9.28 (VD18): now also C8.1, C9.1
- net at U9.3 (XIN): now also Y2.3
- net D4-: now reaches U9.4 (DM4)
- net D4-: now also U8.3 (D-)
- net D4+: now reaches U9.5 (DP4)
- net D4+: now also U8.4 (D+)
- net D3-: now reaches U9.6 (DM3)
- net D3-: now also J11.2 (D-)
- net D3+: now reaches U9.7 (DP3)
- net D3+: now also J11.3 (D+)
- net D2-: now reaches U9.8 (DM2)
- net D2-: now also J10.2 (D-)
- net D2+: now reaches U9.9 (DP2)
- net D2+: now also J10.3 (D+)
- net at U4.18 (OUT17): now also J16.2 (Pin_2)
- net at U4.17 (OUT16): now also J16.4 (Pin_4)
- net at U4.16 (OUT15): now also J16.6 (Pin_6)
- net at U4.15 (OUT14): now also J16.10 (Pin_10)
- net at U4.14 (OUT13): now also J16.12 (Pin_12)
- net at U4.13 (OUT12): now also J16.14 (Pin_14)
- net at U4.12 (OUT11): now also J16.18 (Pin_18)
- net at U4.11 (OUT10): now also J16.20 (Pin_20)
- net at U4.24 (OUT23): now also J16.13 (Pin_13)
- net at U4.10 (OUT9): now also J16.22 (Pin_22)
- net at U4.9 (OUT8): now also J16.26 (Pin_26)
- net at U4.8 (OUT7): now also J16.28 (Pin_28)
- net at U4.7 (OUT6): now also J16.30 (Pin_30)
- net at U4.6 (OUT5): now also J16.34 (Pin_34)
- net at U4.5 (OUT4): now also J16.36 (Pin_36)
- net at U4.4 (OUT3): now also J16.38 (Pin_38)
- net at U4.23 (OUT22): now also J16.11 (Pin_11)
- net at U4.3 (OUT2): now also J16.42 (Pin_42)
- net at U4.2 (OUT1): now also J16.44 (Pin_44)
- net at U4.1 (OUT0): now also J16.46 (Pin_46)
- net at U4.22 (OUT21): now also J16.9 (Pin_9)
- net at U4.21 (OUT20): now also J16.5 (Pin_5)
- net at U4.20 (OUT19): now also J16.3 (Pin_3)
- net at U4.19 (OUT18): now also J16.1 (Pin_1)
- net at U1.25 (IO48): no longer U2.26 (XLAT)
- net at U1.39 (IO1): no longer U2.32 (SIN)
- net MOSI: now reaches U8.10 (PB2)
- net MOSI: now also J3.5 (Pin_5), J3.6 (Pin_6)
- net MISO: now reaches U8.11 (PB3)
- net MISO: now also J3.3 (Pin_3), J3.4 (Pin_4)
- net at U8.16 (XTAL2): now also C3.2, Y1.3
- net at U8.17 (XTAL1): now also C4.2, Y1.1
- net PD0: now reaches U8.18 (PD0)
- net PD0: now also U6.10 (S0), U7.10 (S0)
- net PD1: now reaches U8.19 (PD1)
- net PD1: now also U6.11 (S1), U7.11 (S1)
- net IO4: now reaches U8.20 (PD2)
- net IO4: now also U1.4 (IO4)
- net IO5: now reaches U8.21 (PD3)
- net IO5: now also U1.5 (IO5)
- net PD5: now reaches U8.22 (PD5)
- net PD5: now also U6.15 (~{E})
- net PD4: now reaches U8.25 (PD4)
- net PD4: now also U6.14 (S2), U7.14 (S2)
- net PD6: now reaches U8.26 (PD6)
- net PD6: now also U6.13 (S3), U7.13 (S3)
- net PD7: now reaches U8.27 (PD7)
- net PD7: now also U7.15 (~{E})
- net CS1: now reaches U8.28 (PB4)
- net CS1: now also J3.1 (Pin_1)
- net CS2: now reaches U8.29 (PB5)
- net CS2: now also J3.2 (Pin_2)
- net at U8.42 (AREF): now also C10.1
- net at U8.6 (UCAP): now also C11.1
- net SCK: now reaches U8.9 (PB1)
- net SCK: now also J3.7 (Pin_7), J3.8 (Pin_8)
- net IO8: now reaches U1.12 (IO8)
- net IO38: now reaches U1.31 (IO38)
- net IO38: now also J2.4 (Pin_4)
- net IO39: now reaches U1.32 (IO39)
- net IO39: now also J2.3 (Pin_3)
- net IO42: now reaches U1.35 (IO42)
- net IO42: now also U2.32 (SIN)
- net RXD0: now reaches U1.36 (RXD0)
- net RXD0: now also J9.2 (Pin_2)
- net TXD0: now reaches U1.37 (TXD0)
- net TXD0: now also J9.3 (Pin_3)
- net IO6: now reaches U1.6 (IO6)
- net IO7: now reaches U1.7 (IO7)
- new net EXT_5V: J15.15 (Pin_15), J15.16 (Pin_16), J15.23 (Pin_23), J15.24 (Pin_24), J15.31 (Pin_31), J15.32 (Pin_32), J15.39 (Pin_39), J15.40 (Pin_40), J15.47 (Pin_47), J15.48 (Pin_48), J15.7 (Pin_7), J15.8 (Pin_8), J16.15 (Pin_15), J16.16 (Pin_16), J16.23 (Pin_23), J16.24 (Pin_24), J16.31 (Pin_31), J16.32 (Pin_32), J16.39 (Pin_39), J16.40 (Pin_40), J16.47 (Pin_47), J16.48 (Pin_48), J16.7 (Pin_7), J16.8 (Pin_8), J2.5 (Pin_5), J2.6 (Pin_6), J4.2 (Pin_2), J8.1 (Pin_1), U2.28 (VCC), U3.28 (VCC), U4.28 (VCC)
Other:
- moved on the sheet: C1, C2, C6, J1, R4, R5, U5, U8

Commit message: board
Connections:
- net at U3.1 (OUT0): now also J16.18 (Pin_18); no longer J16.17 (Pin_17)
- net at U3.10 (OUT9): now also J16.42 (Pin_42); no longer J16.41 (Pin_41)
- net at U3.11 (OUT10): now also J16.44 (Pin_44); no longer J16.43 (Pin_43)
- net at U3.12 (OUT11): now also J16.46 (Pin_46); no longer J16.45 (Pin_45)
- net at U3.2 (OUT1): now also J16.20 (Pin_20); no longer J16.19 (Pin_19)
- net at U3.3 (OUT2): now also J16.22 (Pin_22); no longer J16.21 (Pin_21)
- net at U3.4 (OUT3): now also J16.26 (Pin_26); no longer J16.25 (Pin_25)
- net at U3.5 (OUT4): now also J16.28 (Pin_28); no longer J16.27 (Pin_27)
- net at U3.6 (OUT5): now also J16.30 (Pin_30); no longer J16.29 (Pin_29)
- net at U3.7 (OUT6): now also J16.34 (Pin_34); no longer J16.33 (Pin_33)
- net at U3.8 (OUT7): now also J16.36 (Pin_36); no longer J16.35 (Pin_35)
- net at U3.9 (OUT8): now also J16.38 (Pin_38); no longer J16.37 (Pin_37)
- net at U4.1 (OUT0): now also J16.45 (Pin_45); no longer J16.46 (Pin_46)
- net at U4.10 (OUT9): now also J16.21 (Pin_21); no longer J16.22 (Pin_22)
- net at U4.11 (OUT10): now also J16.19 (Pin_19); no longer J16.20 (Pin_20)
- net at U4.12 (OUT11): now also J16.17 (Pin_17); no longer J16.18 (Pin_18)
- net at U4.13 (OUT12): now also J16.13 (Pin_13); no longer J16.14 (Pin_14)
- net at U4.14 (OUT13): now also J16.11 (Pin_11); no longer J16.12 (Pin_12)
- net at J16.10 (Pin_10): now also U4.22 (OUT21); no longer U4.15 (OUT14)
- net at U4.16 (OUT15): now also J16.5 (Pin_5); no longer J16.6 (Pin_6)
- net at U4.17 (OUT16): now also J16.3 (Pin_3); no longer J16.4 (Pin_4)
- net at U4.18 (OUT17): now also J16.1 (Pin_1); no longer J16.2 (Pin_2)
- net at U4.19 (OUT18): now also J16.2 (Pin_2); no longer J16.1 (Pin_1)
- net at U4.2 (OUT1): now also J16.43 (Pin_43); no longer J16.44 (Pin_44)
- net at U4.20 (OUT19): now also J16.4 (Pin_4); no longer J16.3 (Pin_3)
- net at U4.21 (OUT20): now also J16.6 (Pin_6); no longer J16.5 (Pin_5)
- net at J16.9 (Pin_9): now also U4.15 (OUT14); no longer U4.22 (OUT21)
- net at U4.23 (OUT22): now also J16.12 (Pin_12); no longer J16.11 (Pin_11)
- net at U4.24 (OUT23): now also J16.14 (Pin_14); no longer J16.13 (Pin_13)
- net at U4.3 (OUT2): now also J16.41 (Pin_41); no longer J16.42 (Pin_42)
- net at U4.4 (OUT3): now also J16.37 (Pin_37); no longer J16.38 (Pin_38)
- net at U4.5 (OUT4): now also J16.35 (Pin_35); no longer J16.36 (Pin_36)
- net at U4.6 (OUT5): now also J16.33 (Pin_33); no longer J16.34 (Pin_34)
- net at U4.7 (OUT6): now also J16.29 (Pin_29); no longer J16.30 (Pin_30)
- net at U4.8 (OUT7): now also J16.27 (Pin_27); no longer J16.28 (Pin_28)
- net at U4.9 (OUT8): now also J16.25 (Pin_25); no longer J16.26 (Pin_26)

Commit message: duplicated PCB
Parts:
- removed C10, C11, C12, C13, C14, C3, C4: 22pf, Capacitor_SMD:C_0603_1608Metric_Pad1.08x0.95mm_HandSolder, symbol Device:C
- removed U1: ESP32-S3-WROOM-1, RF_Module:ESP32-S3-WROOM-1, symbol RF_Module:ESP32-S3-WROOM-1
- removed U8: ATmega32U4-M, Package_DFN_QFN:QFN-44-1EP_7x7mm_P0.5mm_EP5.2x5.2mm, symbol MCU_Microchip_ATmega:ATmega32U4-M
- removed Y1: Crystal_GND24, Crystal:Crystal_SMD_2520-4Pin_2.5x2.0mm, symbol Device:Crystal_GND24
- added C15, C17, C18, C19, C20, C21, C22, C23, C24: 100nf, Capacitor_SMD:C_0603_1608Metric_Pad1.08x0.95mm_HandSolder, symbol Device:C
- added C16: 2.2uf, Capacitor_SMD:C_0603_1608Metric_Pad1.08x0.95mm_HandSolder, symbol Device:C
- added R10: 5.1k, Resistor_SMD:R_0603_1608Metric_Pad0.98x0.95mm_HandSolder, symbol Device:R_US
- added R11, R12: 27, Resistor_SMD:R_0603_1608Metric_Pad0.98x0.95mm_HandSolder, symbol Device:R_US
- added U1: RP2040, Package_DFN_QFN:QFN-56-1EP_7x7mm_P0.4mm_EP3.2x3.2mm, symbol MCU_RaspberryPi:RP2040
- added U8: W25Q16JVSS, Package_SO:SOIC-8_5.3x5.3mm_P1.27mm, symbol Memory_Flash:W25Q16JVSS
- added Y3: Crystal_GND24, Crystal:Crystal_SMD_2520-4Pin_2.5x2.0mm, symbol Device:Crystal_GND24
Connections:
- net 3.3v: now also C15.1, C16.1, C17.2, C18.2, C19.2, C20.2, C21.2, C22.2, U1.1 (IOVDD), U1.10 (IOVDD), U1.22 (IOVDD), U1.33 (IOVDD), U1.42 (IOVDD), U1.49 (IOVDD), U8.8 (VCC)
- net D1+: now also R12.2
- net D1-: now also R11.2
- net GND: now also C15.2, C16.2, C17.1, C18.1, C19.1, C20.1, C21.1, C22.1, C23.1, C24.2, U1.57 (GND), U8.4 (GND), Y3.2, Y3.4
- net IO39: no longer names the net of J2.3 (Pin_3)
- new net: C23.2, R10.1, Y3.3
- new net: R12.1, U1.47 (USB_DP)
- new net: U1.23 (DVDD), U1.50 (DVDD)
- new net: R11.1, U1.46 (USB_DM)
- new net QSPI_SCLK: U1.52 (QSPI_SCLK), U8.6 (CLK)
- new net QSPI_SD0: U1.53 (QSPI_SD0), U8.5 (DI/IO_{0})
- new net QSPI_SD1: U1.55 (QSPI_SD1), U8.2 (DO/IO_{1})
- new net QSPI_SD2: U1.54 (QSPI_SD2), U8.3 (~{WP}/IO_{2})
- new net QSPI_SD3: U1.51 (QSPI_SD3), U8.7 (~{HOLD}/~{RESET}/IO_{3})
- new net QSPI_SS: U1.56 (~{QSPI_SS}), U8.1 (~{CS})
- new net XIN: C24.1, U1.20 (XIN), Y3.1
- new net XOUT: R10.2, U1.21 (XOUT)

Commit message: refactored gamepads
Parts:
- removed C5, C7, C8, C9: 22pf, Capacitor_SMD:C_0603_1608Metric_Pad1.08x0.95mm_HandSolder, symbol Device:C
- removed J10, J11: USB_A, Connector_USB:USB_A_Molex_67643_Horizontal, symbol Connector:USB_A
- removed R6, R7, R8, R9: 5.1k, Resistor_SMD:R_0603_1608Metric_Pad0.98x0.95mm_HandSolder, symbol Device:R_US
- removed U9: FE1.1s, Package_SO:SSOP-28_3.9x9.9mm_P0.635mm, symbol Interface_USB:FE1.1s
- removed Y2: Crystal_GND24, Crystal:Crystal_SMD_2520-4Pin_2.5x2.0mm, symbol Device:Crystal_GND24
- added H5: (no value), Raspberry-Pi-CM5:RaspberryPi-CM5-Module-Pad, symbol Raspberry-Pi-CM5:RaspberryPi-CM5-Module
Connections:
- net RXD0 is gone; now on net RX0: J9.2 (Pin_2)
- net TXD0 is gone; now on net TX0: J9.3 (Pin_3)
- net TX0: now reaches U1.16 (GPIO13)
- net RX0: now reaches U1.17 (GPIO14)

Commit message: board
Parts:
- removed H5: (no value), Raspberry-Pi-CM5:RaspberryPi-CM5-Module-Pad, symbol Raspberry-Pi-CM5:RaspberryPi-CM5-Module
- added Module1: ComputeModule5-CM5, CM5IO:Raspberry-Pi-5-Compute-Module, symbol CM5IO:ComputeModule5-CM5
- added U9: TS3USB221ARSERG4, RSE10, symbol 2026-06-13_04-03-08:TS3USB221ARSERG4

Commit message: board changes
Parts:
- added J10: Conn_02x06_Odd_Even, Connector_PinHeader_2.54mm:PinHeader_2x06_P2.54mm_Horizontal, symbol Connector_Generic:Conn_02x06_Odd_Even
- added J11, J12: USB_C_Receptacle_USB2.0_16P, Connector_USB:USB_C_Receptacle_GCT_USB4110, symbol Connector:USB_C_Receptacle_USB2.0_16P
- added J13: HDMI_A_1.4, Connector_Video:HDMI_A_Amphenol_10029449-x01xLF_Horizontal, symbol Connector:HDMI_A_1.4
- added J14, J17: USB_C_Receptacle, Connector_USB:USB_C_Receptacle_Amphenol_12401548E4-2A, symbol Connector:USB_C_Receptacle
- added U10: TCA9548AMRGER, Package_DFN_QFN:Texas_RGE0024C_VQFN-24-1EP_4x4mm_P0.5mm_EP2.1x2.1mm, symbol Interface_Expansion:TCA9548AMRGER
Connections:
- net 3.3v: now also J10.10 (Pin_10), J10.9 (Pin_9)
- net CS1: now also J10.1 (Pin_1)
- net CS2: now also J10.2 (Pin_2)
- net GND: now also J10.11 (Pin_11), J10.12 (Pin_12)
- net MISO: now also J10.3 (Pin_3), J10.4 (Pin_4)
- net MOSI: now also J10.5 (Pin_5), J10.6 (Pin_6)
- net SCK: now also J10.7 (Pin_7), J10.8 (Pin_8)
- new net: J11.A1 (GND), J11.A12 (GND), J11.B1 (GND), J11.B12 (GND)
- new net: J11.A4 (VBUS), J11.A9 (VBUS), J11.B4 (VBUS), J11.B9 (VBUS)
- new net: J14.A1 (GND), J14.A12 (GND), J14.B1 (GND), J14.B12 (GND)
- new net: J14.A4 (VBUS), J14.A9 (VBUS), J14.B4 (VBUS), J14.B9 (VBUS)
- new net: J17.A1 (GND), J17.A12 (GND), J17.B1 (GND), J17.B12 (GND)
- new net: J17.A4 (VBUS), J17.A9 (VBUS), J17.B4 (VBUS), J17.B9 (VBUS)
- new net: J12.A1 (GND), J12.A12 (GND), J12.B1 (GND), J12.B12 (GND)
- new net: J12.A4 (VBUS), J12.A9 (VBUS), J12.B4 (VBUS), J12.B9 (VBUS)
