File: PCB/arcade/arcade.kicad_sch (KiCad schematic)
At the start: 52 parts, among them J1 USB_C_Receptacle_USB2.0_16P, J10 Conn_02x06_Odd_Even, J11 USB_C_Receptacle_USB2.0_16P, J12 USB_C_Receptacle_USB2.0_16P, J13 HDMI_A_1.4, J14 USB_C_Receptacle, J15 Conn_02x24_Odd_Even, J16 Conn_02x24_Odd_Even, J17 USB_C_Receptacle, J2 Conn_02x03_Odd_Even, J3 Conn_02x06_Odd_Even, J4 Screw_Terminal_01x02, J5 Screw_Terminal_01x12, J6 Screw_Terminal_01x08, J7 Screw_Terminal_01x12, J8 Conn_01x02_Pin, J9 Conn_01x06_Pin, U1 RP2040, U10 TCA9548AMRGER, U2 TLC5947RHB, U3 TLC5947RHB, U4 TLC5947RHB, U5 ME6211C33M5, U6 CD74HC4067M, U7 CD74HC4067M, U8 W25Q16JVSS, U9 TS3USB221ARSERG4, Y3 Crystal_GND24

Commit message: analog working
Parts:
- removed J10: Conn_02x06_Odd_Even, Connector_PinHeader_2.54mm:PinHeader_2x06_P2.54mm_Horizontal, symbol Connector_Generic:Conn_02x06_Odd_Even
- removed J11, J12: USB_C_Receptacle_USB2.0_16P, Connector_USB:USB_C_Receptacle_GCT_USB4110, symbol Connector:USB_C_Receptacle_USB2.0_16P
- removed J14, J17: USB_C_Receptacle, Connector_USB:USB_C_Receptacle_Amphenol_12401548E4-2A, symbol Connector:USB_C_Receptacle
- added J10: USB3_A_Stacked, Connector_USB:USB3_A_Molex_48406-0001_Horizontal_Stacked, symbol Connector:USB3_A_Stacked
- added J11: USB_A_Stacked, Connector_USB:USB_A_CUI_UJ2-ADH-TH_Horizontal_Stacked, symbol Connector:USB_A_Stacked
