File: PCB/stick2/stick2/stick2.kicad_pcb (KiCad board)
At the start: 2 copper layers, 76 x 63.5 mm, 55 parts, among them J1 Conn_01x04_Pin, J2 Conn_01x16, J3 USB_C_Receptacle_USB2.0_16P, J4 Conn_01x06_Pin, J5 Conn_01x03_Pin, U1 MLX90395xLW, U2 NCP1117ST33T3G, U3 W25Q128JVSIQ, U4 RP2350A, X1 12MHz

Commit message: board changes
Parts:
- moved R5 2.10 mm to (114.2, 86.0)
- moved J2 1.30 mm to (159.0, 99.2)
- moved X1 0.30 mm to (123.5, 95.5)
Connections:
- J4 pad 1: unconnected-(J4-Pin_1-Pad1) -> GND
- J4 pad 2: unconnected-(J4-Pin_2-Pad2) -> VBUS
- J4 pad 3: unconnected-(J4-Pin_3-Pad3) -> +3V3
- J4 pad 4: unconnected-(J4-Pin_4-Pad4) -> /GPIO10
- J4 pad 5: unconnected-(J4-Pin_5-Pad5) -> /GPIO9
- J4 pad 6: unconnected-(J4-Pin_6-Pad6) -> /GPIO8
Routing:
- net +3V3: track 115.1 -> 210.6 mm
- net /GPIO8: track 0.00 -> 82.0 mm
- net /GPIO9: track 0.00 -> 81.5 mm
- net /GPIO10: track 0.00 -> 81.1 mm
- net VBUS: track 159.0 -> 170.0 mm
- net GND: track 58.4 -> 54.3 mm
- net /GPIO22: track 25.7 -> 24.2 mm
- net /COM: track 22.4 -> 20.9 mm
- net /GPIO18: track 17.9 -> 16.5 mm
- net /GPIO24: track 30.7 -> 29.2 mm
- net /GPIO23: track 28.2 -> 26.7 mm
- net /GPIO21: track 24.1 -> 22.7 mm
- net /GPIO15: track 20.6 -> 19.2 mm
- net /GPIO19: track 25.3 -> 24.2 mm
- net /GPIO17: track 24.4 -> 23.2 mm
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