File: PCB/stick2/stick2/stick2.kicad_sch (KiCad schematic)
At the start: 57 parts, among them J1 Conn_01x04_Pin, J2 Conn_01x16, J3 USB_C_Receptacle_USB2.0_16P, J4 Conn_01x06_Pin, J5 Conn_01x03_Pin, SW1 434133025816, SW2 434133025816, U1 MLX90395xLW, U2 NCP1117ST33T3G, U3 W25Q128JVSIQ, U4 RP2350A, X1 12MHz

Commit message: board changes
Connections:
- net +3V3: now also J4.3 (Pin_3)
- net GND: now also J4.1 (Pin_1)
- net GPIO10: now also J4.4 (Pin_4)
- net GPIO8: now also J4.6 (Pin_6)
- net GPIO9: now also J4.5 (Pin_5)
- net VBUS: now also J4.2 (Pin_2)
