File: PCB/stick2/stick2-IO/stick2-IO.kicad_pcb (KiCad board)
At the start: 2 copper layers, 76 x 39 mm, 20 parts, among them J10 Conn_01x12_Pin, J11 Conn_01x04_Pin, J12 Conn_01x05_Pin, J13 Conn_01x16_Pin, J2 Conn_02x04_Row_Letter_Last, J3 Conn_02x04_Row_Letter_Last, J4 Conn_02x04_Row_Letter_Last, J5 Conn_02x04_Row_Letter_Last, J6 Conn_02x04_Row_Letter_Last, J7 Conn_02x04_Row_Letter_Last, J8 Conn_02x04_Row_Letter_Last, J9 Conn_02x04_Row_Letter_Last, U2 TLC5947RHB, U3 TLC5947RHB, U6 CD74HC4067M

Commit message: board changes
Parts:
- moved U6 0.30 mm to (164.0, 76.8)
Routing:
- net Net-(J10-Pin_10): track 87.8 -> 91.8 mm
- net Net-(J10-Pin_11): track 91.4 -> 87.6 mm
- net Net-(J10-Pin_9): track 89.5 -> 87.0 mm
- net Net-(J10-Pin_8): track 92.8 -> 94.4 mm
Other:
- outline, holes or cut-outs redrawn

Commit message: boards
Parts:
- moved H3 0.50 mm to (173.0, 53.0)
- moved H4 0.50 mm to (173.0, 87.0)
- moved H5 0.50 mm to (102.0, 53.0)
- moved H6 0.50 mm to (102.0, 87.0)
- moved J13 0.50 mm to (118.5, 52.0)
Routing:
- net /GND: track 12.7 -> 8.99 mm
Other:
- outline, holes or cut-outs redrawn
